File: 21xt/02-mainbox/mainbox1.0/mainbox1.0.kicad_sch (KiCad schematic)
At the start: 0 parts

Commit message: testing
Other:
- note added: "hihih"
- note removed: "sadfsadfsa"
Changed lines of the file:
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@@
 (kicad_sch (version 20230121) (generator eeschema)
   (paper "A4")
-  (text "sadfsadfsa" (at 58.928 92.583 0)
+  (text "hihih" (at 58.928 92.583 0)
     (effects (font (size 1.27 1.27)) (justify left bottom))
   )

Commit message: teting testing
Other:
- note added: "asdfsadfasd"
- note removed: "hihih"
Changed lines of the file:
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@@
 (kicad_sch (version 20230121) (generator eeschema)
   (paper "A4")
-  (text "hihih" (at 58.928 92.583 0)
+  (text "asdfsadfasd" (at 58.928 92.583 0)
     (effects (font (size 1.27 1.27)) (justify left bottom))
   )

Commit message: sdfsdfsd
Other:
- note added: "sdfsd"
- note removed: "asdfsadfasd"
Changed lines of the file:
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@@
 (kicad_sch (version 20230121) (generator eeschema)
   (paper "A4")
-  (text "asdfsadfasd" (at 58.928 92.583 0)
+  (text "sdfsd" (at 58.928 92.583 0)
     (effects (font (size 1.27 1.27)) (justify left bottom))
   )

Commit message: work please
Other:
- note added: "dddd"
- note removed: "sdfsd"
Changed lines of the file:
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@@
 (kicad_sch (version 20230121) (generator eeschema)
   (paper "A4")
-  (text "sdfsd" (at 58.928 92.583 0)
+  (text "dddd" (at 58.928 92.583 0)
     (effects (font (size 1.27 1.27)) (justify left bottom))
   )

Commit message: yurr
Other:
- note added: "dddddddddd"
- note removed: "dddd"
Changed lines of the file:
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@@
 (kicad_sch (version 20230121) (generator eeschema)
   (paper "A4")
-  (text "dddd" (at 58.928 92.583 0)
+  (text "dddddddddd" (at 58.928 92.583 0)
     (effects (font (size 1.27 1.27)) (justify left bottom))
   )

Commit message: wroking???
Other:
- note added: "sdfsdfsdfsdfsdf"
- note removed: "dddddddddd"
Changed lines of the file:
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@@
 (kicad_sch (version 20230121) (generator eeschema)
   (paper "A4")
-  (text "dddddddddd" (at 58.928 92.583 0)
+  (text "sdfsdfsdfsdfsdf" (at 58.928 92.583 0)
     (effects (font (size 1.27 1.27)) (justify left bottom))
   )

Commit message: idkidk
Other:
- note added: "dfdfdfdf"
- note removed: "sdfsdfsdfsdfsdf"
Changed lines of the file:
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@@
 (kicad_sch (version 20230121) (generator eeschema)
   (paper "A4")
-  (text "sdfsdfsdfsdfsdf" (at 58.928 92.583 0)
+  (text "dfdfdfdf" (at 58.928 92.583 0)
     (effects (font (size 1.27 1.27)) (justify left bottom))
   )

Commit message: Created AD7175-8 file
Other:
- note removed: "dfdfdfdf"
Changed lines of the file:
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@@
 (kicad_sch (version 20230121) (generator eeschema)
   (paper "A4")
-  (text "dfdfdfdf" (at 58.928 92.583 0)
-    (effects (font (size 1.27 1.27)) (justify left bottom))
-  )
   (sheet_instances
     (path "/" (page "1"))
