File: 21xt/02-mainbox/mainbox1.0/StrainGauge_sch.kicad_sch (KiCad schematic)
At the start: 9 parts, among them J4 Conn_01x06, U5 AD8222ACPZ-R7

Commit message: Everything done
Parts:
- removed J4: Conn_01x06, Connector_Molex:Molex_PicoBlade_53047-0610_1x06_P1.25mm_Vertical, symbol Connector_Generic:Conn_01x06
- removed TP14, TP15: TestPoint, TestPoint:TestPoint_Pad_1.5x1.5mm, symbol Connector:TestPoint
- added J1: Conn_01x06, 21xt_footprints:MOLEX_0533980671 (1x6), symbol Connector_Generic:Conn_01x06
Connections:
- net 2.5V: now also J1.1 (Pin_1)
- net GND: now also J1.2 (Pin_2)
- net SG1+: now also J1.3 (Pin_3)
- net SG1-: now also J1.4 (Pin_4)
- net SG2+: now also J1.5 (Pin_5)
- net SG2-: now also J1.6 (Pin_6)
Changed lines of the file:
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@@
   (junction (at 140.97 95.885) (diameter 0) (color 0 0 0 0)
   )
-  (junction (at 138.43 95.885) (diameter 0) (color 0 0 0 0)
-  )
-  (junction (at 153.67 88.265) (diameter 0) (color 0 0 0 0)
-  )
   (junction (at 128.27 79.375) (diameter 0) (color 0 0 0 0)
   )
@@
     (stroke (width 0) (type default))
   )
-  (wire (pts (xy 128.27 95.885) (xy 138.43 95.885))
+  (wire (pts (xy 128.27 95.885) (xy 140.97 95.885))
     (stroke (width 0) (type default))
   )
@@
     (stroke (width 0) (type default))
   )
-  (wire (pts (xy 138.43 95.885) (xy 140.97 95.885))
-    (stroke (width 0) (type default))
-  )
-  (wire (pts (xy 153.67 88.265) (xy 154.305 88.265))
-    (stroke (width 0) (type default))
-  )
   (wire (pts (xy 145.415 86.995) (xy 145.415 88.265))
     (stroke (width 0) (type default))
@@
     (stroke (width 0) (type default))
   )
-  (wire (pts (xy 145.415 88.265) (xy 153.67 88.265))
+  (wire (pts (xy 145.415 88.265) (xy 154.305 88.265))
     (stroke (width 0) (type default))
   )
@@
     )
   )
-  (global_label "SG1-" (shape output) (at 185.42 67.945 180) (fields_autoplaced)
-    (effects (font (size 1.27 1.27)) (justify right))
-    (property "Intersheetrefs" "${INTERSHEET_REFS}" (at 177.1734 67.945 0)
+  (global_label "2.5V" (shape input) (at 210.185 71.755 180) (fields_autoplaced)
+    (effects (font (size 1.27 1.27)) (justify right))
+    (property "Intersheetrefs" "${INTERSHEET_REFS}" (at 203.0874 71.755 0)
+      (effects (font (size 1.27 1.27)) (justify right) hide)
+    )
+  )
+  (global_label "SG1+" (shape output) (at 210.185 76.835 180) (fields_autoplaced)
+    (effects (font (size 1.27 1.27)) (justify right))
+    (property "Intersheetrefs" "${INTERSHEET_REFS}" (at 201.9384 76.835 0)
+      (effects (font (size 1.27 1.27)) (justify right) hide)
+    )
+  )
+  (global_label "SG1-" (shape output) (at 210.185 79.375 180) (fields_autoplaced)
+    (effects (font (size 1.27 1.27)) (justify right))
+    (property "Intersheetrefs" "${INTERSHEET_REFS}" (at 201.9384 79.375 0)
+      (effects (font (size 1.27 1.27)) (justify right) hide)
+    )
+  )
+  (global_label "SG2-" (shape output) (at 210.185 84.455 180) (fields_autoplaced)
+    (effects (font (size 1.27 1.27)) (justify right))
+    (property "Intersheetrefs" "${INTERSHEET_REFS}" (at 201.9384 84.455 0)
+      (effects (font (size 1.27 1.27)) (justify right) hide)
+    )
+  )
+  (global_label "SG2+" (shape output) (at 210.185 81.915 180) (fields_autoplaced)
+    (effects (font (size 1.27 1.27)) (justify right))
+    (property "Intersheetrefs" "${INTERSHEET_REFS}" (at 201.9384 81.915 0)
       (effects (font (size 1.27 1.27)) (justify right) hide)
     )
@@
     )
   )
-  (global_label "SG2+" (shape output) (at 185.42 75.565 180) (fields_autoplaced)
-    (effects (font (size 1.27 1.27)) (justify right))
-    (property "Intersheetrefs" "${INTERSHEET_REFS}" (at 177.1734 75.565 0)
-      (effects (font (size 1.27 1.27)) (justify right) hide)
-    )
-  )
   (global_label "SG2+" (shape input) (at 128.27 104.775 0) (fields_autoplaced)
     (effects (font (size 1.27 1.27)) (justify left))
@@
     )
   )
-  (global_label "SG2-" (shape output) (at 185.42 73.025 180) (fields_autoplaced)
-    (effects (font (size 1.27 1.27)) (justify right))
-    (property "Intersheetrefs" "${INTERSHEET_REFS}" (at 177.1734 73.025 0)
-      (effects (font (size 1.27 1.27)) (justify right) hide)
-    )
-  )
   (global_label "5VADC" (shape input) (at 154.305 88.265 0) (fields_autoplaced)
     (effects (font (size 1.27 1.27)) (justify left))
@@
     )
   )
-  (global_label "SG1+" (shape output) (at 185.42 70.485 180) (fields_autoplaced)
-    (effects (font (size 1.27 1.27)) (justify right))
-    (property "Intersheetrefs" "${INTERSHEET_REFS}" (at 177.1734 70.485 0)
-      (effects (font (size 1.27 1.27)) (justify right) hide)
-    )
-  )
-  (global_label "2.5V" (shape input) (at 185.42 80.645 180) (fields_autoplaced)
-    (effects (font (size 1.27 1.27)) (justify right))
-    (property "Intersheetrefs" "${INTERSHEET_REFS}" (at 178.3224 80.645 0)
-      (effects (font (size 1.27 1.27)) (justify right) hide)
-    )
-  )
   (global_label "SG1-" (shape input) (at 128.27 102.235 0) (fields_autoplaced)
     (effects (font (size 1.27 1.27)) (justify left))
@@
         (path "/fef72a68-b3e4-4609-8f5e-093085beb166/023e5077-10bd-4858-a669-79cb61e1b551"
           (reference "#PWR058") (unit 1)
-        )
-      )
-    )
-  )
-  (symbol (lib_id "Connector:TestPoint") (at 153.67 88.265 0) (unit 1)
-    (in_bom yes) (on_board yes) (dnp no) (fields_autoplaced)
-    (property "Reference" "TP14" (at 156.21 83.693 0)
-      (effects (font (size 1.27 1.27)) (justify left))
-    )
-    (property "Value" "TestPoint" (at 156.21 86.233 0)
-      (effects (font (size 1.27 1.27)) (justify left))
-    )
-    (property "Footprint" "TestPoint:TestPoint_Pad_1.5x1.5mm" (at 158.75 88.265 0)
-      (effects (font (size 1.27 1.27)) hide)
-    )
-    (property "Datasheet" "~" (at 158.75 88.265 0)
-      (effects (font (size 1.27 1.27)) hide)
-    )
-    (pin "1")
-    (instances
-      (project "mainbox1.0"
-        (path "/386ce652-2291-4cad-85a5-fcca6d2077c3/bf4d2e97-bd72-4a0b-a505-9f8ebd51e80b"
-          (reference "TP14") (unit 1)
         )
       )
@@
     )
   )
+  (symbol (lib_id "power:GND") (at 210.185 74.295 270) (unit 1)
+    (in_bom yes) (on_board yes) (dnp no) (fields_autoplaced)
+    (property "Reference" "#PWR01" (at 203.835 74.295 0)
+      (effects (font (size 1.27 1.27)) hide)
+    )
+    (property "Value" "GND" (at 206.375 74.295 90)
+      (effects (font (size 1.27 1.27)) (justify right) hide)
+    )
+    (property "Footprint" "" (at 210.185 74.295 0)
+      (effects (font (size 1.27 1.27)) hide)
+    )
+    (property "Datasheet" "" (at 210.185 74.295 0)
+      (effects (font (size 1.27 1.27)) hide)
+    )
+    (pin "1")
+    (instances
+      (project "mainbox1.0"
+        (path "/386ce652-2291-4cad-85a5-fcca6d2077c3/bf4d2e97-bd72-4a0b-a505-9f8ebd51e80b"
+          (reference "#PWR01") (unit 1)
+        )
+      )
+      (project "Mainboard_priv"
+        (path "/fef72a68-b3e4-4609-8f5e-093085beb166/023e5077-10bd-4858-a669-79cb61e1b551"
+          (reference "#PWR055") (unit 1)
+        )
+      )
+    )
+  )
   (symbol (lib_id "power:GND") (at 142.24 79.375 180) (unit 1)
     (in_bom yes) (on_board yes) (dnp no) (fields_autoplaced)
@@
     )
   )
-  (symbol (lib_id "Connector:TestPoint") (at 138.43 95.885 0) (unit 1)
-    (in_bom yes) (on_board yes) (dnp no) (fields_autoplaced)
-    (property "Reference" "TP15" (at 140.97 91.313 0)
-      (effects (font (size 1.27 1.27)) (justify left))
-    )
-    (property "Value" "TestPoint" (at 140.97 93.853 0)
-      (effects (font (size 1.27 1.27)) (justify left))
-    )
-    (property "Footprint" "TestPoint:TestPoint_Pad_1.5x1.5mm" (at 143.51 95.885 0)
-      (effects (font (size 1.27 1.27)) hide)
-    )
-    (property "Datasheet" "~" (at 143.51 95.885 0)
-      (effects (font (size 1.27 1.27)) hide)
-    )
-    (pin "1")
-    (instances
-      (project "mainbox1.0"
-        (path "/386ce652-2291-4cad-85a5-fcca6d2077c3/bf4d2e97-bd72-4a0b-a505-9f8ebd51e80b"
-          (reference "TP15") (unit 1)
-        )
-      )
-    )
-  )
-  (symbol (lib_id "power:GND") (at 185.42 78.105 270) (unit 1)
-    (in_bom yes) (on_board yes) (dnp no) (fields_autoplaced)
-    (property "Reference" "#PWR048" (at 179.07 78.105 0)
-      (effects (font (size 1.27 1.27)) hide)
-    )
-    (property "Value" "GND" (at 181.61 78.105 90)
-      (effects (font (size 1.27 1.27)) (justify right) hide)
-    )
-    (property "Footprint" "" (at 185.42 78.105 0)
-      (effects (font (size 1.27 1.27)) hide)
-    )
-    (property "Datasheet" "" (at 185.42 78.105 0)
-      (effects (font (size 1.27 1.27)) hide)
-    )
-    (pin "1")
-    (instances
-      (project "mainbox1.0"
-        (path "/386ce652-2291-4cad-85a5-fcca6d2077c3/bf4d2e97-bd72-4a0b-a505-9f8ebd51e80b"
-          (reference "#PWR048") (unit 1)
-        )
-      )
-      (project "Mainboard_priv"
-        (path "/fef72a68-b3e4-4609-8f5e-093085beb166/023e5077-10bd-4858-a669-79cb61e1b551"
-          (reference "#PWR055") (unit 1)
-        )
-      )
-    )
-  )
   (symbol (lib_id "power:GND") (at 140.97 103.505 0) (unit 1)
     (in_bom yes) (on_board yes) (dnp no) (fields_autoplaced)
@@
     )
   )
-  (symbol (lib_id "Connector_Generic:Conn_01x06") (at 190.5 73.025 0) (unit 1)
-    (in_bom yes) (on_board yes) (dnp no) (fields_autoplaced)
-    (property "Reference" "J4" (at 193.675 73.025 0)
-      (effects (font (size 1.27 1.27)) (justify left))
-    )
-    (property "Value" "Conn_01x06" (at 193.675 75.565 0)
-      (effects (font (size 1.27 1.27)) (justify left))
-    )
-    (property "Footprint" "Connector_Molex:Molex_PicoBlade_53047-0610_1x06_P1.25mm_Vertical" (at 190.5 73.025 0)
-      (effects (font (size 1.27 1.27)) hide)
-    )
-    (property "Datasheet" "~" (at 190.5 73.025 0)
+  (symbol (lib_id "Connector_Generic:Conn_01x06") (at 215.265 76.835 0) (unit 1)
+    (in_bom yes) (on_board yes) (dnp no) (fields_autoplaced)
+    (property "Reference" "J1" (at 218.44 76.835 0)
+      (effects (font (size 1.27 1.27)) (justify left))
+    )
+    (property "Value" "Conn_01x06" (at 218.44 79.375 0)
+      (effects (font (size 1.27 1.27)) (justify left))
+    )
+    (property "Footprint" "21xt_footprints:MOLEX_0533980671 (1x6)" (at 215.265 76.835 0)
+      (effects (font (size 1.27 1.27)) hide)
+    )
+    (property "Datasheet" "~" (at 215.265 76.835 0)
       (effects (font (size 1.27 1.27)) hide)
     )
@@
       (project "mainbox1.0"
         (path "/386ce652-2291-4cad-85a5-fcca6d2077c3/bf4d2e97-bd72-4a0b-a505-9f8ebd51e80b"
-          (reference "J4") (unit 1)
-        )
-      )
+          (reference "J1") (unit 1)
+        )
+      )

Commit message: shift SSD
Parts:
- J1: footprint 21xt_footprints:MOLEX_0533980671 (1x6) -> (none)
Changed lines of the file:
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@@
       (effects (font (size 1.27 1.27)) (justify left))
     )
-    (property "Footprint" "21xt_footprints:MOLEX_0533980671 (1x6)" (at 215.265 76.835 0)
+    (property "Footprint" "" (at 215.265 76.835 0)
       (effects (font (size 1.27 1.27)) hide)
     )
