File: 21xt/03-wireless_strain_gauge/PumpDACBreakout/Untitled.kicad_sch (KiCad schematic)
At the start: 19 parts, among them IC1 AD5721RBRUZ, J1 Conn_01x06, J2 Conn_01x01

Commit message: updates
Parts:
- R5: footprint Resistor_SMD:R_0402_1005Metric_Pad0.72x0.64mm_HandSolder -> Resistor_SMD:R_0603_1608Metric
Changed lines of the file:
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@@
       (effects (font (size 1.27 1.27)))
     )
-    (property "Footprint" "Resistor_SMD:R_0402_1005Metric_Pad0.72x0.64mm_HandSolder" (at 80.772 81.915 90)
+    (property "Footprint" "Resistor_SMD:R_0603_1608Metric" (at 80.772 81.915 90)
       (effects (font (size 1.27 1.27)) hide)
     )
