File: 21xt/03-wireless_strain_gauge/PumpDACBreakout/_autosave-Untitled.kicad_pcb (KiCad board)
At the start: 2 copper layers, 24.5 x 17.3 mm, 13 parts, among them J1 Conn_01x06, J2 Conn_01x01

Commit message: updates
Routing:
- net Sclk: track 0.00 -> 15.9 mm
- net Sync': track 0.00 -> 14.3 mm
- net MOSI: track 0.41 -> 12.7 mm
- net Vin: track 20.0 -> 31.3 mm
- net MISO: track 0.33 -> 10.9 mm
- net GND: vias 18 -> 19
Changed lines of the file:
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@@
       (outputformat 1)
       (mirror false)
-      (drillshape 1)
+      (drillshape 0)
       (scaleselection 1)
       (outputdirectory "")
@@
   (via (at 116.2 78.2975) (size 0.8) (drill 0.4) (layers "F.Cu" "B.Cu") (net 5))
   (via (at 119.2 83.7775) (size 0.8) (drill 0.4) (layers "F.Cu" "B.Cu") (net 5))
+  (via (at 124.54 86.75) (size 0.8) (drill 0.4) (layers "F.Cu" "B.Cu") (free) (net 5))
   (via (at 118.94 81.19) (size 0.4) (drill 0.1) (layers "F.Cu" "B.Cu") (net 5))
   (via (at 119.53 81.19) (size 0.4) (drill 0.1) (layers "F.Cu" "B.Cu") (net 5))
@@
   (segment (start 120.19 81.9825) (end 120.21 82.0025) (width 0.25) (layer "F.Cu") (net 8))
   (segment (start 118.265 80.9575) (end 118.29 80.9825) (width 0.3) (layer "F.Cu") (net 8))
+  (segment (start 123.01 84.2175) (end 122.42 83.6275) (width 0.3) (layer "F.Cu") (net 8))
+  (segment (start 122.42 89.26) (end 123.01 88.67) (width 0.3) (layer "F.Cu") (net 8))
   (segment (start 120.775 81.9825) (end 121.5 82.7075) (width 0.25) (layer "F.Cu") (net 8))
   (segment (start 120.19 81.9825) (end 120.775 81.9825) (width 0.25) (layer "F.Cu") (net 8))
   (segment (start 113.7725 80.9575) (end 118.265 80.9575) (width 0.3) (layer "F.Cu") (net 8))
+  (segment (start 123.01 84.755) (end 123.01 88.67) (width 0.25) (layer "F.Cu") (net 8))
+  (segment (start 122.42 83.6275) (end 121.5 82.7075) (width 0.3) (layer "F.Cu") (net 8))
+  (segment (start 123.01 88.67) (end 123.01 84.2175) (width 0.3) (layer "F.Cu") (net 8))
   (via (at 113.61 81.12) (size 0.8) (drill 0.4) (layers "F.Cu" "B.Cu") (net 8))
   (segment (start 122.42 89.26) (end 119.34 89.26) (width 0.3) (layer "B.Cu") (net 8))
@@
   (segment (start 119.34 89.26) (end 113.61 83.53) (width 0.3) (layer "B.Cu") (net 8))
   (segment (start 130.42 89.26) (end 130.42 88.948528) (width 0.4) (layer "F.Cu") (net 10))
+  (segment (start 130.01 81.26) (end 130.845 80.425) (width 0.4) (layer "F.Cu") (net 10))
+  (segment (start 130.845 80.425) (end 132.43 80.425) (width 0.4) (layer "F.Cu") (net 10))
+  (segment (start 130.42 88.948528) (end 130 88.528528) (width 0.4) (layer "F.Cu") (net 10))
   (segment (start 130 86.225584) (end 130.01 86.215584) (width 0.4) (layer "F.Cu") (net 10))
+  (segment (start 130.01 86.215584) (end 130.01 81.26) (width 0.4) (layer "F.Cu") (net 10))
+  (segment (start 130 88.528528) (end 130 86.225584) (width 0.4) (layer "F.Cu") (net 10))
+  (segment (start 129.41 85.967056) (end 129.41 80.517056) (width 0.4) (layer "F.Cu") (net 12))
   (segment (start 128.42 89.26) (end 128.71 88.97) (width 0.4) (layer "F.Cu") (net 12))
+  (segment (start 128.71 86.667056) (end 129.41 85.967056) (width 0.4) (layer "F.Cu") (net 12))
+  (segment (start 128.71 88.97) (end 128.71 86.667056) (width 0.4) (layer "F.Cu") (net 12))
+  (segment (start 130.802056 79.125) (end 132.43 79.125) (width 0.4) (layer "F.Cu") (net 12))
+  (segment (start 129.41 80.517056) (end 130.802056 79.125) (width 0.4) (layer "F.Cu") (net 12))
+  (segment (start 128.81 85.718528) (end 128.81 80.268528) (width 0.4) (layer "F.Cu") (net 13))
+  (segment (start 128.81 80.268528) (end 130.603528 78.475) (width 0.4) (layer "F.Cu") (net 13))
+  (segment (start 126.42 88.108528) (end 128.81 85.718528) (width 0.4) (layer "F.Cu") (net 13))
+  (segment (start 126.42 89.26) (end 126.42 88.108528) (width 0.4) (layer "F.Cu") (net 13))
+  (segment (start 130.603528 78.475) (end 132.43 78.475) (width 0.4) (layer "F.Cu") (net 13))
+  (segment (start 128.21 85.47) (end 128.21 80.02) (width 0.4) (layer "F.Cu") (net 14))
+  (segment (start 124.42 89.26) (end 128.21 85.47) (width 0.4) (layer "F.Cu") (net 14))
+  (segment (start 130.405 77.825) (end 132.43 77.825) (width 0.4) (layer "F.Cu") (net 14))
+  (segment (start 128.21 80.02) (end 130.405 77.825) (width 0.4) (layer "F.Cu") (net 14))
   (segment (start 120.835 80.9825) (end 121.31 80.5075) (width 0.25) (layer "F.Cu") (net 15))
   (segment (start 120.19 80.9825) (end 120.835 80.9825) (width 0.25) (layer "F.Cu") (net 15))
