File: 21xt/03-wireless_strain_gauge/PumpDACBreakout/Untitled.kicad_pcb (KiCad board)
At the start: 2 copper layers, 1 part, among them IC1 AD5721RBRUZ

Commit message: updates
Parts:
- removed IC1: AD5721RBRUZ, 21xt_footprints:SOP65P640X120-16N
- added 10k: 10k, Resistor_SMD:R_0402_1005Metric_Pad0.72x0.64mm_HandSolder, F.Cu at (117.2, 83.4)
- added 1u (10v): 1u (10V), Resistor_SMD:R_0402_1005Metric, F.Cu at (116.0, 82.1)
- added 4.7u: 4.7u, Resistor_SMD:R_0402_1005Metric, F.Cu at (117.7, 78.3)
- added 4.7u: 4.7u, Resistor_SMD:R_0402_1005Metric, F.Cu at (121.3, 81.0)
- added 55k: 55k, Resistor_SMD:R_0402_1005Metric_Pad0.72x0.64mm_HandSolder, F.Cu at (119.2, 79.4)
- added Bip-DAC (AD5761R): AD5721RBRUZ, 21xt_footprints:AD5721, F.Cu at (129.6, 78.8)
- added C1: 10u, Resistor_SMD:R_0402_1005Metric, F.Cu at (125.1, 77.4)
- added C4: 2.2u, Resistor_SMD:R_0402_1005Metric, F.Cu at (121.5, 83.2)
- added J1: Conn_01x06, Connector_PinHeader_2.00mm:PinHeader_1x06_P2.00mm_Vertical, F.Cu at (132.4, 89.3)
- added J2: Conn_01x01, Connector_PinHeader_2.00mm:PinHeader_1x01_P2.00mm_Vertical, F.Cu at (121.9, 76.8)
- added PS1: LM27762DSSR, 21xt_footprints:LM27762DSST, F.Cu at (119.2, 81.7)
- added R2: 10k, Resistor_SMD:R_0402_1005Metric_Pad0.72x0.64mm_HandSolder, F.Cu at (120.2, 84.7)
- added R5: 172k, Resistor_SMD:R_0603_1608Metric, F.Cu at (116.2, 79.9)
Routing:
- net Vin: track 0.00 -> 31.3 mm, vias 0 -> 1
- net GND: track 0.00 -> 22.5 mm, vias 0 -> 20
- net Sclk: track 0.00 -> 15.9 mm
- net Sync': track 0.00 -> 14.3 mm
- net -5v: track 0.00 -> 13.7 mm
- net MOSI: track 0.00 -> 12.7 mm
- net MISO: track 0.00 -> 10.9 mm
- net Net-(PS1-FB-): track 0.00 -> 2.72 mm
- net Net-(PS1-C1+): track 0.00 -> 2.54 mm
- net Net-(PS1-FB+): track 0.00 -> 2.43 mm
- net Net-(PS1-C1-): track 0.00 -> 2.33 mm
- net Net-(IC1-VREFIN/VREFOUT): track 0.00 -> 1.82 mm
- net Net-(PS1-CP): track 0.00 -> 1.32 mm
- net Net-(PS1-OUT+): track 0.00 -> 1.26 mm
- added copper zone on B.Cu, net GND
- added copper zone on F.Cu, net GND
Other:
- board outline added: 24.5 x 17.3 mm
- board text added: "10/11/2024"
- board text added: "10k"
- board text added: "10u"
- board text added: "172k"
- board text added: "2.2u"
- board text added: "5v"
- board text added: "Bip. DAC + Inv. Charge Pump"
- board text added: "Blue Jay Racing -- breakout"
- board text added: "Clk"
- board text added: "GND"
- board text added: "MISO"
- board text added: "MOSI"
- board text added: "Sync'"
