File: 21xt/big_hbridge/big_hbridge.kicad_pcb (KiCad board)
At the start: 4 copper layers, 82.5 x 63.5 mm, 30 parts, among them J1 Screw_Terminal_01x02, J2 Screw_Terminal_01x02, J4 Barrel_Jack, J5 Conn_01x06, Q1 NMOS, Q2 NMOS, Q3 NMOS, Q4 NMOS, U1 LTC7061EMSE-PBF

Commit message: gerber export, should figure this out
Parts:
- C1, C2: value 1uF -> .1uF
- moved H6 0.10 mm to (43.2, 22.1)
Other:
- outline, holes or cut-outs redrawn
