File: 21xt/big_hbridge/big_hbridge.kicad_sch (KiCad schematic)
At the start: 31 parts, among them J1 Screw_Terminal_01x02, J2 Screw_Terminal_01x02, J4 Barrel_Jack, J5 Conn_01x06, Q1 NMOS, Q2 NMOS, Q3 NMOS, Q4 NMOS, U1 LTC7061EMSE-PBF

Commit message: gerber export, should figure this out
Parts:
- removed C3: 1uF, big_hbridge_fp:CAPPA3050W60L1050D500, symbol Device:C_Polarized
- C1, C2: value 1uF -> .1uF
Other:
- note removed: "MAL202139108E3"
Changed lines of the file:
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@@
 		)
 	)
-	(text "MAL202139108E3"
-		(exclude_from_sim no)
-		(at 198.628 29.972 0)
-		(effects
-			(font
-				(size 1.27 1.27)
-			)
-		)
-	)
 	(global_label "VCC"
 		(shape input)
@@
 		)
 	)
-	(global_label "VIN"
-		(shape input)
-		(at 181.61 27.94 90)
-		(fields_autoplaced yes)
-		(effects
-			(font
-				(size 1.27 1.27)
-			)
-			(justify left)
-		)
-		(property "Intersheetrefs" "${INTERSHEET_REFS}"
-			(at 181.61 21.9309 90)
-			(effects
-				(font
-					(size 1.27 1.27)
-				)
-				(justify left)
-				(hide yes)
-			)
-		)
-	)
 	(global_label "VCC"
 		(shape input)
@@
 			)
 		)
-		(property "Value" "1uF"
+		(property "Value" ".1uF"
 			(at 160.02 144.78 90)
 			(effects
@@
 	)
 	(symbol
-		(lib_id "Device:C_Polarized")
-		(at 181.61 31.75 0)
-		(unit 1)
-		(exclude_from_sim no)
-		(in_bom yes)
-		(on_board yes)
-		(dnp no)
-		(fields_autoplaced yes)
-		(property "Reference" "C3"
-			(at 185.42 29.5909 0)
-			(effects
-				(font
-					(size 1.27 1.27)
-				)
-				(justify left)
-			)
-		)
-		(property "Value" "1uF"
-			(at 185.42 32.1309 0)
-			(effects
-				(font
-					(size 1.27 1.27)
-				)
-				(justify left)
-			)
-		)
-		(property "Footprint" "big_hbridge_fp:CAPPA3050W60L1050D500"
-			(at 182.5752 35.56 0)
-			(effects
-				(font
-					(size 1.27 1.27)
-				)
-				(hide yes)
-			)
-		)
-		(property "Datasheet" "~"
-			(at 181.61 31.75 0)
-			(effects
-				(font
-					(size 1.27 1.27)
-				)
-				(hide yes)
-			)
-		)
-		(property "Description" "Polarized capacitor"
-			(at 181.61 31.75 0)
-			(effects
-				(font
-					(size 1.27 1.27)
-				)
-				(hide yes)
-			)
-		)
-		(pin "2"
-		)
-		(pin "1"
-		)
-		(instances
-			(project ""
-				(path "/22e7b83c-d1c3-430a-908d-ecad4a096a4c"
-					(reference "C3")
-					(unit 1)
-				)
-			)
-		)
-	)
-	(symbol
 		(lib_id "Device:R")
 		(at 29.21 96.52 90)
@@
 			)
 		)
-		(property "Value" "1uF"
+		(property "Value" ".1uF"
 			(at 161.29 88.9 90)
 			(effects
@@
 					(unit 1)
 				)
-			)
-		)
-	)
-	(symbol
-		(lib_id "power:GNDPWR")
-		(at 181.61 35.56 0)
-		(unit 1)
-		(exclude_from_sim no)
-		(in_bom yes)
-		(on_board yes)
-		(dnp no)
-		(fields_autoplaced yes)
-		(property "Reference" "#PWR06"
-			(at 181.61 40.64 0)
-			(effects
-				(font
-					(size 1.27 1.27)
-				)
-				(hide yes)
-			)
-		)
-		(property "Value" "GNDPWR"
-			(at 181.483 39.37 0)
-			(effects
-				(font
-					(size 1.27 1.27)
-				)
-			)
-		)
-		(property "Footprint" ""
-			(at 181.61 36.83 0)
-			(effects
-				(font
-					(size 1.27 1.27)
-				)
-				(hide yes)
-			)
-		)
-		(property "Datasheet" ""
-			(at 181.61 36.83 0)
-			(effects
-				(font
-					(size 1.27 1.27)
-				)
-				(hide yes)
-			)
-		)
-		(property "Description" "Power symbol creates a global label with name \"GNDPWR\" , global ground"
-			(at 181.61 35.56 0)
-			(effects
-				(font
-					(size 1.27 1.27)
-				)
-				(hide yes)
-			)
-		)
-		(pin "1"
-		)
-		(instances
-			(project "big_hbridge"
-				(path "/22e7b83c-d1c3-430a-908d-ecad4a096a4c"
-					(reference "#PWR06")
-					(unit 1)
-				)
