File: 21xt/02-mainbox/mainbox2.0/XBee.kicad_sch (KiCad schematic)
At the start: 13 parts, among them IC1 XBP9X-DMUS-011, J3 Conn_01x02, J4 Conn_01x02

Commit message: sophie needs to fix this
Parts:
- removed J4: Conn_01x02, Connector_PinHeader_2.54mm:PinHeader_1x02_P2.54mm_Vertical, symbol Connector_Generic:Conn_01x02
- PS1: footprint 21xt_footprints:R78B5015L - -> 21xt_footprints:CONV_R-78B3.3-1.5
Changed lines of the file:
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@@
     (effects (font (size 1.27 1.27)) (justify left bottom))
-  )
-  (global_label "DINXBee" (shape input) (at 90.805 143.51 0) (fields_autoplaced)
-    (effects (font (size 1.27 1.27)) (justify left))
-    (property "Intersheetrefs" "${INTERSHEET_REFS}" (at 101.6522 143.51 0)
-      (effects (font (size 1.27 1.27)) (justify left) hide)
-    )
   )
   (global_label "DOUTXBee" (shape output) (at 173.99 71.12 180) (fields_autoplaced)
@@
     )
   )
-  (global_label "DOUTXBee" (shape input) (at 90.805 140.97 0) (fields_autoplaced)
-    (effects (font (size 1.27 1.27)) (justify left))
-    (property "Intersheetrefs" "${INTERSHEET_REFS}" (at 103.3455 140.97 0)
-      (effects (font (size 1.27 1.27)) (justify left) hide)
-    )
-  )
   (symbol (lib_id "power:GND") (at 106.68 81.28 180) (unit 1)
     (in_bom yes) (on_board yes) (dnp no) (fields_autoplaced)
@@
       (effects (font (size 1.27 1.27)) (justify left))
     )
-    (property "Footprint" "21xt_footprints:R78B5015L -" (at 4.14 110.49 0)
+    (property "Footprint" "21xt_footprints:CONV_R-78B3.3-1.5" (at 4.14 110.49 0)
       (effects (font (size 1.27 1.27)) (justify left top) hide)
     )
@@
         )
       )
-    )
-  )
-  (symbol (lib_id "Connector_Generic:Conn_01x02") (at 85.725 143.51 180) (unit 1)
-    (in_bom yes) (on_board yes) (dnp no) (fields_autoplaced)
-    (property "Reference" "J4" (at 85.725 135.255 0)
-      (effects (font (size 1.27 1.27)))
-    )
-    (property "Value" "Conn_01x02" (at 85.725 137.795 0)
-      (effects (font (size 1.27 1.27)))
-    )
-    (property "Footprint" "Connector_PinHeader_2.54mm:PinHeader_1x02_P2.54mm_Vertical" (at 85.725 143.51 0)
-      (effects (font (size 1.27 1.27)) hide)
-    )
-    (property "Datasheet" "~" (at 85.725 143.51 0)
-      (effects (font (size 1.27 1.27)) hide)
-    )
-    (pin "1")
-    (pin "2")
-    (instances
-      (project "mainbox1.0"
-        (path "/386ce652-2291-4cad-85a5-fcca6d2077c3/dd0157a9-838c-4507-b641-fb16517bbb6e"
-          (reference "J4") (unit 1)
-        )
-      )
-      (project "mainbox2.0"
-        (path "/f7ca7218-80bf-4776-ba9d-a28b83375023/5d6e883b-1bc0-4ce9-8a5a-9d01f2a447ea"
-          (reference "J6") (unit 1)
-        )
-      )
-      (project "Mainboard_priv"
-        (path "/fef72a68-b3e4-4609-8f5e-093085beb166/ccbaf9e4-0c9b-47b5-a316-0ae6750baa2c"
-          (reference "J1") (unit 1)
-        )
-      )

Commit message: schematic check
Other:
- moved on the sheet: TP3
Changed lines of the file:
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@@
   (junction (at 112.395 88.9) (diameter 0) (color 0 0 0 0)
   )
+  (junction (at 143.51 88.9) (diameter 0) (color 0 0 0 0)
+  )
   (junction (at 128.905 88.9) (diameter 0) (color 0 0 0 0)
   )
@@
   )
   (junction (at 106.68 88.9) (diameter 0) (color 0 0 0 0)
-  )
-  (junction (at 147.955 88.9) (diameter 0) (color 0 0 0 0)
   )
   (no_connect (at 237.49 71.12))
@@
     (stroke (width 0) (type default))
   )
-  (wire (pts (xy 147.955 88.9) (xy 154.305 88.9))
-    (stroke (width 0) (type default))
-  )
   (wire (pts (xy 251.46 81.28) (xy 251.46 83.185))
     (stroke (width 0) (type default))
@@
     (stroke (width 0) (type default))
   )
-  (wire (pts (xy 128.905 88.9) (xy 147.955 88.9))
+  (wire (pts (xy 128.905 88.9) (xy 143.51 88.9))
+    (stroke (width 0) (type default))
+  )
+  (wire (pts (xy 143.51 88.9) (xy 154.305 88.9))
     (stroke (width 0) (type default))
   )
@@
     )
   )
-  (symbol (lib_id "Connector:TestPoint") (at 147.955 88.9 0) (unit 1)
-    (in_bom yes) (on_board yes) (dnp no) (fields_autoplaced)
-    (property "Reference" "TP3" (at 150.495 84.328 0)
+  (symbol (lib_id "Connector:TestPoint") (at 143.51 88.9 0) (unit 1)
+    (in_bom yes) (on_board yes) (dnp no)
+    (property "Reference" "TP3" (at 144.145 83.82 0)
       (effects (font (size 1.27 1.27)) (justify left))
     )
-    (property "Value" "TestPoint" (at 150.495 86.868 0)
-      (effects (font (size 1.27 1.27)) (justify left))
-    )
-    (property "Footprint" "TestPoint:TestPoint_Pad_1.5x1.5mm" (at 153.035 88.9 0)
-      (effects (font (size 1.27 1.27)) hide)
-    )
-    (property "Datasheet" "~" (at 153.035 88.9 0)
-      (effects (font (size 1.27 1.27)) hide)
-    )
+    (property "Value" "TestPoint" (at 144.78 86.995 0)
+      (effects (font (size 1.27 1.27)) (justify left) hide)
+    )
+    (property "Footprint" "TestPoint:TestPoint_Pad_1.5x1.5mm" (at 148.59 88.9 0)
+      (effects (font (size 1.27 1.27)) hide)
+    )
+    (property "Datasheet" "~" (at 148.59 88.9 0)
+      (effects (font (size 1.27 1.27)) hide)
+    )

Commit message: schematic markups minus pcie
Other:
- note added: "isnt this guy really large"
- note added: "should label voltage somehow"
- note added: "which of these grounds do we need to connect"
Changed lines of the file:
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@@
     (stroke (width 0) (type default))
+  )
+  (arc (start 307.34 52.07) (mid 249.8709 101.9127) (end 173.99 96.52)
+    (stroke (width 0) (type default))
+    (fill (type none))
+  )
+  (arc (start 307.34 52.07) (mid 282.5641 92.8344) (end 236.22 104.14)
+    (stroke (width 0) (type default))
+    (fill (type none))
+  )
+  (arc (start 307.34 52.07) (mid 283.8792 96.0094) (end 236.22 110.49)
+    (stroke (width 0) (type default))
+    (fill (type none))
+  )
+  (arc (start 307.34 52.07) (mid 248.8188 99.3727) (end 173.99 91.44)
+    (stroke (width 0) (type default))
+    (fill (type none))
+  )
+  (arc (start 151.13 -10.16) (mid 176.9626 25.2646) (end 170.18 68.58)
+    (stroke (width 0) (type default))
+    (fill (type none))
+  )
+  (arc (start 307.34 52.07) (mid 243.5583 86.6727) (end 173.99 66.04)
+    (stroke (width 0) (type default))
+    (fill (type none))
+  )
+  (arc (start 307.34 52.07) (mid 276.3604 76.0615) (end 237.49 71.12)
+    (stroke (width 0) (type default))
+    (fill (type none))
+  )
+  (arc (start -26.67 116.84) (mid 31.7691 83.71) (end 96.52 101.6)
+    (stroke (width 0) (type default))
+    (fill (type none))
+  )
+  (text "isnt this guy really large" (at -55.88 115.57 0)
+    (effects (font (size 1.27 1.27)) (justify left bottom))
   )
   (text "xbee" (at 203.2 55.245 0)
     (effects (font (size 1.27 1.27)) (justify left bottom))
   )
+  (text "which of these grounds do we need to connect" (at 308.61 53.34 0)
+    (effects (font (size 1.27 1.27)) (justify left bottom))
+  )
+  (text "should label voltage somehow" (at 127 -8.89 0)
+    (effects (font (size 1.27 1.27)) (justify left bottom))
+  )

Commit message: progress
Parts:
- removed TP16, TP3: TestPoint, TestPoint:TestPoint_Pad_1.5x1.5mm, symbol Connector:TestPoint
- C27: value 4.7 -> 4.7uF
- C28: value 0.1 -> 0.1uF
Connections:
- net GND: now also IC1.11 (GND_2), IC1.13 (GND_3), IC1.22 (GND_4), IC1.35 (GND_5)
- net VOUT renamed 3V3_XBEE
- no-connect marks 31 -> 27
Other:
- note added: "Looking at a few alternative smaller chips"
- note removed: "isnt this guy really large"
- note removed: "should label voltage somehow"
- note removed: "which of these grounds do we need to connect"
- moved on the sheet: C26, C27, C28, C29, C30, C31, L1, PS1
