File: 21xt/02-mainbox/mainbox2.0ac/PCIe.kicad_sch (KiCad schematic)
At the start: 20 parts, among them IC6 AP3441LSHE-7B, J3 Conn_01x16, J5 MDT275M02001, Q1 DMG1012T-7

Commit message: board cope
Connections:
- net 5.2V: no longer J3.15 (Pin_15), J3.16 (Pin_16), R4.1
- net GNDS: now also J3.11 (Pin_11), J3.14 (Pin_14), J3.5 (Pin_5), J3.8 (Pin_8), R2.1
- net PCIE_RST_B_SW: now also R2.2; no longer R2.1
- removed net GND: J3.11 (Pin_11), J3.14 (Pin_14), J3.5 (Pin_5), J3.8 (Pin_8), R2.2
- new net 5V PCIE: J3.15 (Pin_15), J3.16 (Pin_16), R4.1
Other:
- moved on the sheet: J3
