File: 21xt/02-mainbox/mainbox2.0ac/mainbox2.0.kicad_pcb (KiCad board)
At the start: 4 copper layers, 88.8 x 56 mm, 69 parts, among them IC1 SN74LVC2T45DCTTG4, IC2 XBP9X-DMUS-011, IC6 AP3441LSHE-7B, IC7 SN74LVC2T45DCTTG4, IC8 SN74LVC2T45DCTTG4, J1 Conn_01x10, J10 Conn_02x20_Odd_Even, J3 Conn_01x16, J4 Conn_01x01_Pin, J5 MDT275M02001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

Commit message: board cope
Parts:
- moved C25 22.4 mm to (127.9, 67.0), turned to 0 degrees
- moved C26 20.2 mm to (127.9, 68.2), turned to 0 degrees
- moved R15 18.0 mm to (63.5, 90.0), turned to 90 degrees
- moved R2 17.9 mm to (68.6, 87.2)
- moved C41 16.9 mm to (83.0, 89.5)
- moved R10 16.1 mm to (66.4, 89.4)
- moved Q1 16.1 mm to (68.4, 89.6)
- moved C16 15.3 mm to (129.8, 97.4)
- moved L1 15.2 mm to (125.2, 70.6)
- moved C45 15.1 mm to (136.6, 97.4)
- moved C40 14.7 mm to (83.0, 90.6)
- moved J6 14.0 mm to (75.0, 78.2), turned to 180 degrees
- moved IC1 11.6 mm to (133.2, 105.6)
- moved C14 9.18 mm to (129.8, 106.7)
- moved C44 6.68 mm to (129.8, 101.3)
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Connections:
- C11 pad 1: GNDD -> GNDA
- C14 pad 1: GNDD -> GNDA
- C15 pad 1: GNDD -> GNDA
- C16 pad 1: GNDD -> GNDA
- C25 pad 2: GNDD -> GNDA
- C26 pad 2: GNDD -> GNDA
- C27 pad 1: GNDD -> GNDA
- C28 pad 1: GNDD -> GNDA
- C29 pad 1: GNDD -> GNDA
- C3 pad 1: GNDD -> GNDA
- C30 pad 1: GNDD -> GNDA
- C36 pad 2: GNDS -> GNDA
- C37 pad 2: GNDS -> GNDA
- C4 pad 1: GNDD -> GNDA
- C40 pad 2: GNDS -> GNDA
- C41 pad 2: GNDS -> GNDA
- C42 pad 2: GNDS -> GNDA
- C43 pad 2: GNDS -> GNDA
- C44 pad 1: GNDD -> GNDA
- C45 pad 1: GNDD -> GNDA
- C46 pad 1: GNDD -> GNDA
- IC1 pad 4: GNDD -> GNDA
- IC1 pad 5: GNDD -> GNDA
- IC2 pad 1: GNDD -> GNDA
- IC2 pad 11: GNDD -> GNDA
- IC2 pad 13: GNDD -> GNDA
- IC2 pad 22: GNDD -> GNDA
- IC2 pad 35: GNDD -> GNDA
- IC6 pad 4: GNDS -> GNDA
- IC6 pad 8: GNDS -> GNDA
- IC6 pad 9: GNDS -> GNDA
- IC7 pad 4: GNDD -> GNDA
- IC7 pad 5: GNDD -> GNDA
- IC8 pad 4: GNDD -> GNDA
- IC8 pad 5: GNDD -> GNDA
- J1 pad 8: GNDD -> GNDA
- J10 pad 14: GNDD -> GNDA
- J10 pad 20: GNDD -> GNDA
- J10 pad 25: GNDD -> GNDA
- J10 pad 30: GNDD -> GNDA
- J10 pad 34: GNDD -> GNDA
- J10 pad 6: GNDD -> GNDA
- J10 pad 9: GNDD -> GNDA
- J3 pad 11: GND -> GNDA
- J3 pad 14: GND -> GNDA
- J3 pad 15: 5.2V -> 5V PCIE
- J3 pad 16: 5.2V -> 5V PCIE
- J3 pad 5: GND -> GNDA
- J3 pad 8: GND -> GNDA
- J5 pad 1: GNDS -> GNDA
- J5 pad 15: GNDS -> GNDA
- J5 pad 21: GNDS -> GNDA
- J5 pad 27: GNDS -> GNDA
- J5 pad 3: GNDS -> GNDA
- J5 pad 33: GNDS -> GNDA
- J5 pad 39: GNDS -> GNDA
- J5 pad 45: GNDS -> GNDA
- J5 pad 51: GNDS -> GNDA
- J5 pad 57: GNDS -> GNDA
- J5 pad 71: GNDS -> GNDA
- J5 pad 73: GNDS -> GNDA
- J5 pad 75: GNDS -> GNDA
- J5 pad 9: GNDS -> GNDA
- J5 pad MP1: GNDS -> GNDA
- J5 pad MP2: GNDS -> GNDA
- J6 pad 1: GNDD -> GNDA
- J8 pad 12: GNDD -> GNDA
- PS1 pad 2: GNDD -> GNDA
- PS2 pad 1: GNDD -> GNDA
- PS2 pad 5: GNDD -> GNDA
- R12 pad 1: GNDS -> GNDA
- R15 pad 2: GNDS -> GNDA
- R2 pad 1: PCIE_RST_B_SW -> GNDA
- R2 pad 2: GND -> PCIE_RST_B_SW
- R4 pad 1: 5.2V -> 5V PCIE
- R8 pad 2: GNDS -> GNDA
- U1 pad 15: GNDD -> GNDA
- U1 pad 17: GNDD -> GNDA
Routing:
- net GNDA: track 30.3 -> 109.4 mm, vias 8 -> 249
- net 3V3: track 6.28 -> 72.9 mm, vias 0 -> 5
- net IN1(3.3V): track 70.8 -> 18.8 mm, vias 0 -> 1
- net IN2(3.3V): track 65.6 -> 21.7 mm, vias 0 -> 1
- net GNDD: track 38.3 -> 0.00 mm, vias 15 -> 0
- net 5V PCIE: track 0.00 -> 25.6 mm, vias 0 -> 2
- net GNDS: track 22.0 -> 0.00 mm, vias 91 -> 0
- net Net-(J3-Pin_1): track 25.6 -> 6.44 mm, vias 2 -> 0
- net DIGITAL_OUTPUT_1: track 52.3 -> 37.4 mm
- net DIGITAL_OUTPUT_2: track 54.8 -> 43.6 mm
- net 3V3_XBEE: track 42.9 -> 53.9 mm
- net Net-(IC6-FB): track 1.98 -> 11.5 mm
- net IN2(5V): track 5.03 -> 13.0 mm
- net VCC3V3: track 10.2 -> 3.34 mm
- net 5.2V: track 30.1 -> 36.1 mm, vias 8 -> 9
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- added copper zone on B.Cu, net 3V3
- added copper zone on In2.Cu, net GNDA
- removed copper zone on In1.Cu, net GNDS
Other:
- outline, holes or cut-outs redrawn
