File: 21xt/main_bulkhead/main_bulkhead.kicad_pcb (KiCad board)
At the start: 4 copper layers, 65 x 38 mm, 30 parts, among them J1 GIGABLOX_NANO_SWITCH_REVA_MOD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, J11 2337822-2, J2 90816-0008, J3 T4041017041-000, J4 T4041017041-000, J5 Conn_01x02_Pin, J9 2337822-2, T1 749013011, T2 749013011

Commit message: resized
Parts:
- moved J5 66.3 mm to (4.23, 37.5), turned to 0 degrees
- moved C2 48.5 mm to (47.1, 27.1)
- moved R5 46.6 mm to (43.5, 33.9), turned to 0 degrees
- moved R8 46.1 mm to (43.5, 30.4), turned to 0 degrees
- moved R6 42.3 mm to (43.5, 32.7), turned to 0 degrees
- moved R7 38.5 mm to (43.5, 31.6), turned to 0 degrees
- moved R12 32.5 mm to (14.9, 26.4), turned to 90 degrees
- moved R11 32.3 mm to (16.4, 26.4), turned to 90 degrees
- moved T1 31.9 mm to (16.3, 34.1), turned to 90 degrees
- moved C8 31.7 mm to (16.7, 22.8), turned to 90 degrees
- moved C4 30.7 mm to (43.0, 27.9)
- moved J2 30.2 mm to (55.1, 35.0), turned to 0 degrees
- moved J9 25.2 mm to (32.9, 32.4), turned to 180 degrees
- moved J11 17.5 mm to (55.6, 11.1), turned to 180 degrees
- moved C6 16.7 mm to (19.7, 25.4), turned to 90 degrees
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Connections:
- J1 pad 21: unconnected-(J1-P1D_N-Pad21) -> P1D_N
- J1 pad 22: unconnected-(J1-P0D_N-Pad22) -> P0D_N
- J1 pad 23: unconnected-(J1-P1D_P-Pad23) -> P1D_P
- J1 pad 24: unconnected-(J1-P0D_P-Pad24) -> P0D_P
- J1 pad 25: unconnected-(J1-P1C_N-Pad25) -> P1C_N
- J1 pad 26: unconnected-(J1-P0C_N-Pad26) -> P0C_N
- J1 pad 27: unconnected-(J1-P1C_P-Pad27) -> P1C_P
- J1 pad 28: unconnected-(J1-P0C_P-Pad28) -> P0C_P
- J10 pad 1: M3C_N -> M0C_N
- J10 pad 2: M3C_P -> M0C_P
- J10 pad 3: M3D_P -> M0D_P
- J10 pad 4: M3D_N -> M0D_N
- J10 pad 5: M3B_P -> M0B_P
- J10 pad 6: M3B_N -> M0B_N
- J10 pad 7: M3A_P -> M0A_P
- J10 pad 8: M3A_N -> M0A_N
- J11 pad 11: P3D_P -> P0D_P
- J11 pad 12: P3D_N -> P0D_N
- J11 pad 13: M3D_N -> M0D_N
- J11 pad 14: M3D_P -> M0D_P
- J11 pad 16: M3C_N -> M0C_N
- J11 pad 17: M3C_P -> M0C_P
- J11 pad 19: M3B_N -> M0B_N
- J11 pad 2: P3A_P -> P0A_P
- J11 pad 20: M3B_P -> M0B_P
- J11 pad 22: M3A_N -> M0A_N
- J11 pad 23: M3A_P -> M0A_P
- J11 pad 3: P3A_N -> P0A_N
- J11 pad 5: P3B_P -> P0B_P
- J11 pad 6: P3B_N -> P0B_N
- J11 pad 8: P3C_P -> P0C_P
- J11 pad 9: P3C_N -> P0C_N
- J2 pad 1: M2A_P -> M3A_P
- J2 pad 2: M2A_N -> M3A_N
- J2 pad 3: M2B_P -> M3B_P
- J2 pad 4: M2B_N -> M3B_N
- J2 pad 5: M2C_P -> M3C_P
- J2 pad 6: M2C_N -> M3C_N
- J2 pad 7: M2D_P -> M3D_P
- J2 pad 8: M2D_N -> M3D_N
- J3 pad 1: M0A_P -> M2A_P
- J3 pad 2: M0A_N -> M2A_N
- J3 pad 3: M0B_P -> M2B_P
- J3 pad 4: M0B_N -> M2B_N
- J9 pad 11: P2D_P -> P3D_P
- J9 pad 12: P2D_N -> P3D_N
- J9 pad 13: M2D_N -> M3D_N
- J9 pad 14: M2D_P -> M3D_P
- J9 pad 16: M2C_N -> M3C_N
- J9 pad 17: M2C_P -> M3C_P
- J9 pad 19: M2B_N -> M3B_N
- J9 pad 2: P2A_P -> P3A_P
- J9 pad 20: M2B_P -> M3B_P
- J9 pad 22: M2A_N -> M3A_N
- J9 pad 23: M2A_P -> M3A_P
- J9 pad 3: P2A_N -> P3A_N
- J9 pad 5: P2B_P -> P3B_P
- J9 pad 6: P2B_N -> P3B_N
- J9 pad 8: P2C_P -> P3C_P
- J9 pad 9: P2C_N -> P3C_N
- T1 pad 1: P0B_P -> P2B_P
- T1 pad 11: M0A_P -> M2A_P
- T1 pad 14: M0B_N -> M2B_N
- T1 pad 16: M0B_P -> M2B_P
- T1 pad 3: P0B_N -> P2B_N
- T1 pad 6: P0A_P -> P2A_P
- T1 pad 8: P0A_N -> P2A_N
- T1 pad 9: M0A_N -> M2A_N
Routing:
- net M0B_P: track 61.2 -> 2.94 mm, vias 1 -> 0
- net M0B_N: track 58.9 -> 4.22 mm, vias 1 -> 0
- net M2A_P: track 64.0 -> 13.8 mm, vias 2 -> 0
- net M2C_N: track 49.6 -> 0.00 mm, vias 2 -> 0
- net M2C_P: track 48.8 -> 0.00 mm, vias 2 -> 0
- net M2A_N: track 64.1 -> 16.9 mm, vias 2 -> 0
- net M2D_N: track 46.7 -> 0.00 mm, vias 2 -> 0
- net M2B_N: track 53.7 -> 10.3 mm, vias 2 -> 0
- net M2B_P: track 53.8 -> 10.6 mm, vias 2 -> 0
- net M0A_N: track 58.5 -> 16.7 mm
- net M0A_P: track 60.0 -> 19.0 mm
- net M2D_P: track 40.7 -> 0.00 mm, vias 2 -> 0
- net P0C_N: track 0.00 -> 37.0 mm
- net P0C_P: track 0.00 -> 37.0 mm
- net P0D_P: track 0.00 -> 34.2 mm
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Other:
- board size 65 x 38 mm -> 65 x 42 mm
- board text added: "1"
- board text added: "2"
- board text added: "3"
- board text added: "4"
- board text added: "5"
- board text added: "5v"
- board text added: "6"
- board text added: "7"
- board text added: "8"
- board text added: "A+"
- board text added: "A-"
- board text added: "AN"
- board text added: "AP"
- board text added: "B+"
- board text added: "B-"
- board text added: "BN"
- board text added: "BP"
- board text added: "C+"
- board text added: "C-"
- board text added: "CN"
- board text added: "CP"
- board text added: "D+"
- board text added: "D-"
- board text added: "DN"
- board text added: "DP"
- board text added: "black"
- board text added: "blue"
- board text added: "brown"
- board text added: "gnd"
- board text added: "green"
- board text added: "orange"
- board text added: "pblade"
- board text added: "pflex"
- board text added: "purple"
- board text added: "red"
- board text added: "yellow"

Commit message: finished silkscreening
Connections:
- J2 pad 1: M3A_P -> M3C_N
- J2 pad 2: M3A_N -> M3C_P
- J2 pad 3: M3B_P -> M3D_P
- J2 pad 4: M3B_N -> M3D_N
- J2 pad 5: M3C_P -> M3B_P
- J2 pad 6: M3C_N -> M3B_N
- J2 pad 7: M3D_P -> M3A_P
- J2 pad 8: M3D_N -> M3A_N
Routing:
- net M3B_P: track 21.9 -> 33.4 mm
- net M3C_P: track 37.1 -> 31.7 mm, vias 0 -> 2
- net M3A_P: track 26.9 -> 22.9 mm
- net M3C_N: track 33.9 -> 37.6 mm, vias 0 -> 2
- net M3B_N: track 26.4 -> 29.0 mm
- net M3D_P: track 44.3 -> 43.0 mm, vias 0 -> 2
- net M3A_N: track 28.8 -> 29.8 mm
- net M3D_N: track 41.0 -> 40.5 mm, vias 0 -> 2
Other:
- board text added: "RX"
- board text added: "TX"
- board text added: "b"
- board text added: "br"
- board text added: "g"
- board text added: "m12"
- board text added: "o"
- board text added: "rj45"
- board text added: "tia/eia 568A"
- board text added: "wb"
- board text added: "wbr"
- board text added: "wg"
- board text added: "wo"

Commit message: Main ethernet bulkhead merge (#12)
Co-authored-by: Sophie Noureddine <sophienoureddine6@gmail.com>
Routing:
- net M2A_N: track 16.9 -> 17.7 mm
Changed lines of the file:
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@@
     (fp_arc (start -1.7 7.275) (mid -8 0.975) (end -1.7 -5.325)
       (stroke (width 0.1) (type solid)) (layer "B.Fab"))
-    (pad "1" thru_hole rect locked (at 0 0 180) (size 1.3 1.3) (drill 0.8) (layers "*.Cu" "*.Mask")
+    (pad "1" thru_hole rect locked (at 0 0 180) (size 1.5 1.5) (drill 1.1) (layers "*.Cu" "*.Mask")
       (net 42 "M1B_P") (pinfunction "1") (pintype "passive"))
-    (pad "2" thru_hole circle locked (at -0.625 1.95 180) (size 1.3 1.3) (drill 0.8) (layers "*.Cu" "*.Mask")
+    (pad "2" thru_hole circle locked (at -0.625 1.95 180) (size 1.5 1.5) (drill 1.1) (layers "*.Cu" "*.Mask")
       (net 43 "M1B_N") (pinfunction "2") (pintype "passive"))
-    (pad "3" thru_hole circle locked (at -3.4 0 180) (size 1.3 1.3) (drill 0.8) (layers "*.Cu" "*.Mask")
+    (pad "3" thru_hole circle locked (at -3.4 0 180) (size 1.5 1.5) (drill 1.1) (layers "*.Cu" "*.Mask")
       (net 44 "M1A_P") (pinfunction "3") (pintype "passive"))
-    (pad "4" thru_hole circle locked (at -2.775 1.95 180) (size 1.3 1.3) (drill 0.8) (layers "*.Cu" "*.Mask")
+    (pad "4" thru_hole circle locked (at -2.775 1.95 180) (size 1.5 1.5) (drill 1.1) (layers "*.Cu" "*.Mask")
       (net 45 "M1A_N") (pinfunction "4") (pintype "passive"))
     (model ":DESKTOP_PCB:c-t4041017041-000-a-3d.stp"
@@
     (fp_arc (start -1.7 7.275) (mid -8 0.975) (end -1.7 -5.325)
       (stroke (width 0.1) (type solid)) (layer "B.Fab"))
-    (pad "1" thru_hole rect locked (at 0 0 180) (size 1.3 1.3) (drill 0.8) (layers "*.Cu" "*.Mask")
+    (pad "1" thru_hole rect locked (at 0 0 180) (size 1.5 1.5) (drill 1.1) (layers "*.Cu" "*.Mask")
       (net 34 "M2A_P") (pinfunction "1") (pintype "passive"))
-    (pad "2" thru_hole circle locked (at -0.625 1.95 180) (size 1.3 1.3) (drill 0.8) (layers "*.Cu" "*.Mask")
+    (pad "2" thru_hole circle locked (at -0.625 1.95 180) (size 1.5 1.5) (drill 1.1) (layers "*.Cu" "*.Mask")
       (net 35 "M2A_N") (pinfunction "2") (pintype "passive"))
-    (pad "3" thru_hole circle locked (at -3.4 0 180) (size 1.3 1.3) (drill 0.8) (layers "*.Cu" "*.Mask")
+    (pad "3" thru_hole circle locked (at -3.4 0 180) (size 1.3 1.3) (drill 1.1) (layers "*.Cu" "*.Mask")
       (net 36 "M2B_P") (pinfunction "3") (pintype "passive"))
-    (pad "4" thru_hole circle locked (at -2.775 1.95 180) (size 1.3 1.3) (drill 0.8) (layers "*.Cu" "*.Mask")
+    (pad "4" thru_hole circle locked (at -2.775 1.95 180) (size 1.5 1.5) (drill 1.1) (layers "*.Cu" "*.Mask")
       (net 37 "M2B_N") (pinfunction "4") (pintype "passive"))
     (model ":DESKTOP_PCB:c-t4041017041-000-a-3d.stp"
@@
   (via (at 26.62 17.35) (size 0.5) (drill 0.3) (layers "F.Cu" "B.Cu") (net 33))
   (via (at 26.78 18.41) (size 0.5) (drill 0.3) (layers "F.Cu" "B.Cu") (net 33))
-  (segment (start 5.56 27.421353) (end 5.56 28.605) (width 0.127) (layer "F.Cu") (net 34))
+  (segment (start 6.26921 26.32) (end 5.56 27.02921) (width 0.127) (layer "F.Cu") (net 34))
+  (segment (start 11.95 32.22) (end 10.868 32.22) (width 0.127) (layer "F.Cu") (net 34))
+  (segment (start 10.868 32.22) (end 10.7195 32.0715) (width 0.127) (layer "F.Cu") (net 34))
+  (segment (start 5.56 27.02921) (end 5.56 28.605) (width 0.127) (layer "F.Cu") (net 34))
   (segment (start 5.56 28.605) (end 6.225 29.27) (width 0.127) (layer "F.Cu") (net 34))
-  (segment (start 9.338647 26.47) (end 6.511353 26.47) (width 0.127) (layer "F.Cu") (net 34))
-  (segment (start 10.7195 32.0715) (end 10.7195 27.850853) (width 0.127) (layer "F.Cu") (net 34))
-  (segment (start 10.7195 27.850853) (end 9.338647 26.47) (width 0.127) (layer "F.Cu") (net 34))
-  (segment (start 10.868 32.22) (end 10.7195 32.0715) (width 0.127) (layer "F.Cu") (net 34))
-  (segment (start 11.95 32.22) (end 10.868 32.22) (width 0.127) (layer "F.Cu") (net 34))
-  (segment (start 6.511353 26.47) (end 5.56 27.421353) (width 0.127) (layer "F.Cu") (net 34))
-  (segment (start 5.394 30.12) (end 7.056 30.12) (width 0.127) (layer "F.Cu") (net 35))
-  (segment (start 5.306 27.284) (end 5.306 30.032) (width 0.127) (layer "F.Cu") (net 35))
+  (segment (start 10.7195 27.6195) (end 9.42 26.32) (width 0.127) (layer "F.Cu") (net 34))
+  (segment (start 9.42 26.32) (end 6.26921 26.32) (width 0.127) (layer "F.Cu") (net 34))
+  (segment (start 10.7195 32.0715) (end 10.7195 27.6195) (width 0.127) (layer "F.Cu") (net 34))
+  (segment (start 5.41 30.28) (end 7.06 30.28) (width 0.127) (layer "F.Cu") (net 35))
+  (segment (start 5.24 30.11) (end 5.41 30.28) (width 0.127) (layer "F.Cu") (net 35))
+  (segment (start 9.5 26.02) (end 6.21 26.02) (width 0.127) (layer "F.Cu") (net 35))
+  (segment (start 7.06 30.28) (end 7.38 29.96) (width 0.127) (layer "F.Cu") (net 35))
   (segment (start 7.38 27.85) (end 6.85 27.32) (width 0.127) (layer "F.Cu") (net 35))
-  (segment (start 11.95 28.722143) (end 9.247857 26.02) (width 0.127) (layer "F.Cu") (net 35))
-  (segment (start 11.95 29.68) (end 11.95 28.722143) (width 0.127) (layer "F.Cu") (net 35))
-  (segment (start 9.247857 26.02) (end 6.57 26.02) (width 0.127) (layer "F.Cu") (net 35))
-  (segment (start 6.57 26.02) (end 5.306 27.284) (width 0.127) (layer "F.Cu") (net 35))
-  (segment (start 7.38 29.796) (end 7.38 27.85) (width 0.127) (layer "F.Cu") (net 35))
-  (segment (start 7.056 30.12) (end 7.38 29.796) (width 0.127) (layer "F.Cu") (net 35))
-  (segment (start 5.306 30.032) (end 5.394 30.12) (width 0.127) (layer "F.Cu") (net 35))
+  (segment (start 7.38 29.96) (end 7.38 27.85) (width 0.127) (layer "F.Cu") (net 35))
+  (segment (start 6.21 26.02) (end 5.24 26.99) (width 0.127) (layer "F.Cu") (net 35))
+  (segment (start 11.95 28.47) (end 9.5 26.02) (width 0.127) (layer "F.Cu") (net 35))
+  (segment (start 11.95 29.68) (end 11.95 28.47) (width 0.127) (layer "F.Cu") (net 35))
+  (segment (start 5.24 26.99) (end 5.24 30.11) (width 0.127) (layer "F.Cu") (net 35))
   (segment (start 10.15 37.405) (end 10.15 29.795) (width 0.127) (layer "F.Cu") (net 36))
   (segment (start 11.95 38.57) (end 11.315 38.57) (width 0.127) (layer "F.Cu") (net 36))
@@
   (segment (start 10.86 10.185) (end 9.625 8.95) (width 0.254) (layer "F.Cu") (net 44))
   (segment (start 10.86 13.98) (end 10.86 10.185) (width 0.254) (layer "F.Cu") (net 44))
-  (segment (start 13.4 13.98) (end 13.4 11.4) (width 0.254) (layer "F.Cu") (net 45))
-  (segment (start 13.4 11.4) (end 9 7) (width 0.254) (layer "F.Cu") (net 45))
+  (segment (start 13.4 13.98) (end 13.4 11.04) (width 0.254) (layer "F.Cu") (net 45))
+  (segment (start 13.4 11.04) (end 9.36 7) (width 0.254) (layer "F.Cu") (net 45))
+  (segment (start 9.36 7) (end 9 7) (width 0.254) (layer "F.Cu") (net 45))
   (segment (start 52.475 24.858447) (end 52.475 18.72) (width 0.127) (layer "F.Cu") (net 46))
   (segment (start 55.527348 26.496582) (end 54.113135 26.496582) (width 0.127) (layer "F.Cu") (net 46))

Commit message: m
Routing:
- net M2B_N: track 10.3 -> 21.5 mm
Changed lines of the file:
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@@
     (pad "2" thru_hole circle locked (at -0.625 1.95 180) (size 1.5 1.5) (drill 1.1) (layers "*.Cu" "*.Mask")
       (net 35 "M2A_N") (pinfunction "2") (pintype "passive"))
-    (pad "3" thru_hole circle locked (at -3.4 0 180) (size 1.3 1.3) (drill 1.1) (layers "*.Cu" "*.Mask")
+    (pad "3" thru_hole circle locked (at -3.4 0 180) (size 1.5 1.5) (drill 1.1) (layers "*.Cu" "*.Mask")
       (net 36 "M2B_P") (pinfunction "3") (pintype "passive"))
     (pad "4" thru_hole circle locked (at -2.775 1.95 180) (size 1.5 1.5) (drill 1.1) (layers "*.Cu" "*.Mask")
@@
   (segment (start 11.95 29.68) (end 11.95 28.47) (width 0.127) (layer "F.Cu") (net 35))
   (segment (start 5.24 26.99) (end 5.24 30.11) (width 0.127) (layer "F.Cu") (net 35))
-  (segment (start 10.15 37.405) (end 10.15 29.795) (width 0.127) (layer "F.Cu") (net 36))
-  (segment (start 11.95 38.57) (end 11.315 38.57) (width 0.127) (layer "F.Cu") (net 36))
-  (segment (start 11.315 38.57) (end 10.15 37.405) (width 0.127) (layer "F.Cu") (net 36))
+  (segment (start 10.15 37.71) (end 10.15 29.795) (width 0.127) (layer "F.Cu") (net 36))
   (segment (start 10.15 29.795) (end 9.625 29.27) (width 0.127) (layer "F.Cu") (net 36))
-  (segment (start 10.4655 35.1805) (end 10.4655 28.7855) (width 0.127) (layer "F.Cu") (net 37))
-  (segment (start 11.95 36.03) (end 11.315 36.03) (width 0.127) (layer "F.Cu") (net 37))
-  (segment (start 11.315 36.03) (end 10.4655 35.1805) (width 0.127) (layer "F.Cu") (net 37))
-  (segment (start 10.4655 28.7855) (end 9 27.32) (width 0.127) (layer "F.Cu") (net 37))
+  (segment (start 11.01 38.57) (end 10.15 37.71) (width 0.127) (layer "F.Cu") (net 36))
+  (segment (start 11.95 38.57) (end 11.01 38.57) (width 0.127) (layer "F.Cu") (net 36))
+  (segment (start 12.966 37.93) (end 13.16 38.124) (width 0.127) (layer "F.Cu") (net 37))
+  (segment (start 10.59 37.63) (end 10.89 37.93) (width 0.127) (layer "F.Cu") (net 37))
+  (segment (start 10.59 36.88) (end 10.59 37.63) (width 0.127) (layer "F.Cu") (net 37))
+  (segment (start 8.53 36.93) (end 8.53 27.79) (width 0.127) (layer "F.Cu") (net 37))
+  (segment (start 13.16 39) (end 13 39.16) (width 0.127) (layer "F.Cu") (net 37))
+  (segment (start 8.53 27.79) (end 9 27.32) (width 0.127) (layer "F.Cu") (net 37))
+  (segment (start 13 39.16) (end 10.76 39.16) (width 0.127) (layer "F.Cu") (net 37))
+  (segment (start 11.44 36.03) (end 10.59 36.88) (width 0.127) (layer "F.Cu") (net 37))
+  (segment (start 13.16 38.124) (end 13.16 39) (width 0.127) (layer "F.Cu") (net 37))
+  (segment (start 10.76 39.16) (end 8.53 36.93) (width 0.127) (layer "F.Cu") (net 37))
+  (segment (start 10.89 37.93) (end 12.966 37.93) (width 0.127) (layer "F.Cu") (net 37))
+  (segment (start 11.95 36.03) (end 11.44 36.03) (width 0.127) (layer "F.Cu") (net 37))
   (segment (start 61.365 20.425) (end 61.365 18.72) (width 0.127) (layer "F.Cu") (net 38))
   (segment (start 61.45 20.51) (end 61.365 20.425) (width 0.127) (layer "F.Cu") (net 38))
