File: 21xt/dyno_inst/inputprot.kicad_sch (KiCad schematic)
At the start: 23 parts, among them U1 1SS362FV_L3F, U10 ADA4945-1ACPZ-R2, U2 1SS362FV_L3F, U4 1SS362FV_L3F, U9 1SS362FV_L3F

Commit message: ye
Parts:
- removed R10, R9: 19.1k, symbol Device:R
- removed R5, R6: 1.78k, symbol Device:R
- removed R7, R8: 38.3, symbol Device:R
- removed U10: ADA4945-1ACPZ-R2, LFCSP16_ADA4945-1ACPZ-R2_ADI, symbol dyno_inst_sym:ADA4945-1ACPZ-R2
Connections:
- net -DCSIG^: now reaches CR4.2, R4.2
- net +DCSIG^: now reaches CR3.2, R3.2
Other:
- note removed: "R9-R12, <=1%"

Commit message: sche
Connections:
- net +2v5exc is gone; now on net +5vexc: U1.2 (C2), U2.2 (C2), U4.2 (C2), U9.2 (C2)
- net -2v5exc is gone; now on net -5vexc: U1.1 (A1), U2.1 (A1), U4.1 (A1), U9.1 (A1)
- net +DCEX renamed +DCEXC
- net -DCEX renamed -DCEXC
Other:
- note removed: "Rf"
- note removed: "Rg"
Changed lines of the file:
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@@
-		)
-	)
-	(text "Rf"
-		(exclude_from_sim no)
-		(at 104.648 31.75 0)
-		(effects
-			(font
-				(size 1.27 1.27)
-			)
-		)
-	)
-	(text "Rg"
-		(exclude_from_sim no)
-		(at 89.916 44.196 0)
-		(effects
-			(font
-				(size 1.27 1.27)
-			)
 		)
 	)
@@
 		)
 	)
-	(text "Rg"
-		(exclude_from_sim no)
-		(at 90.424 29.718 0)
-		(effects
-			(font
-				(size 1.27 1.27)
-			)
-		)
-	)
-	(text "Rf"
-		(exclude_from_sim no)
-		(at 103.632 42.418 0)
-		(effects
-			(font
-				(size 1.27 1.27)
-			)
-		)
-	)
 	(global_label "-DCSIG^"
 		(shape output)
@@
 		)
 	)
-	(global_label "+2v5exc"
+	(global_label "+5vexc"
 		(shape input)
 		(at 48.26 78.74 90)
@@
 		)
 		(property "Intersheetrefs" "${INTERSHEET_REFS}"
-			(at 48.26 67.5905 90)
+			(at 48.26 68.8 90)
 			(effects
 				(font
@@
 		)
 	)
-	(global_label "-DCEX"
+	(global_label "-DCEXC"
 		(shape output)
 		(at 27.94 87.63 180)
@@
 		)
 		(property "Intersheetrefs" "${INTERSHEET_REFS}"
-			(at 18.4839 87.63 0)
-			(effects
-				(font
-					(size 1.27 1.27)
-				)
-				(justify right)
-				(hide yes)
-			)
-		)
-	)
-	(global_label "+DCEX"
+			(at 17.2139 87.63 0)
+			(effects
+				(font
+					(size 1.27 1.27)
+				)
+				(justify right)
+				(hide yes)
+			)
+		)
+	)
+	(global_label "+DCEXC"
 		(shape output)
 		(at 27.94 85.09 180)
@@
 		)
 		(property "Intersheetrefs" "${INTERSHEET_REFS}"
-			(at 18.4839 85.09 0)
-			(effects
-				(font
-					(size 1.27 1.27)
-				)
-				(justify right)
-				(hide yes)
-			)
-		)
-	)
-	(global_label "+2v5exc"
+			(at 17.2139 85.09 0)
+			(effects
+				(font
+					(size 1.27 1.27)
+				)
+				(justify right)
+				(hide yes)
+			)
+		)
+	)
+	(global_label "+5vexc"
 		(shape input)
 		(at 45.72 29.21 90)
@@
 		)
 		(property "Intersheetrefs" "${INTERSHEET_REFS}"
-			(at 45.72 18.0605 90)
-			(effects
-				(font
-					(size 1.27 1.27)
-				)
-				(justify left)
-				(hide yes)
-			)
-		)
-	)
-	(global_label "-2v5exc"
+			(at 45.72 19.27 90)
+			(effects
+				(font
+					(size 1.27 1.27)
+				)
+				(justify left)
+				(hide yes)
+			)
+		)
+	)
+	(global_label "-5vexc"
 		(shape input)
 		(at 50.8 29.21 90)
@@
 		)
 		(property "Intersheetrefs" "${INTERSHEET_REFS}"
-			(at 50.8 18.0605 90)
-			(effects
-				(font
-					(size 1.27 1.27)
-				)
-				(justify left)
-				(hide yes)
-			)
-		)
-	)
-	(global_label "-2v5exc"
+			(at 50.8 19.27 90)
+			(effects
+				(font
+					(size 1.27 1.27)
+				)
+				(justify left)
+				(hide yes)
+			)
+		)
+	)
+	(global_label "-5vexc"
 		(shape input)
 		(at 48.26 93.98 270)
@@
 		)
 		(property "Intersheetrefs" "${INTERSHEET_REFS}"
-			(at 48.26 105.1295 90)
-			(effects
-				(font
-					(size 1.27 1.27)
-				)
-				(justify right)
-				(hide yes)
-			)
-		)
-	)
-	(global_label "-2v5exc"
+			(at 48.26 103.92 90)
+			(effects
+				(font
+					(size 1.27 1.27)
+				)
+				(justify right)
+				(hide yes)
+			)
+		)
+	)
+	(global_label "-5vexc"
 		(shape input)
 		(at 45.72 44.45 270)
@@
 		)
 		(property "Intersheetrefs" "${INTERSHEET_REFS}"
-			(at 45.72 55.5995 90)
-			(effects
-				(font
-					(size 1.27 1.27)
-				)
-				(justify right)
-				(hide yes)
-			)
-		)
-	)
-	(global_label "+2v5exc"
+			(at 45.72 54.39 90)
+			(effects
+				(font
+					(size 1.27 1.27)
+				)
+				(justify right)
+				(hide yes)
+			)
+		)
+	)
+	(global_label "+5vexc"
 		(shape input)
 		(at 50.8 44.45 270)
@@
 		)
 		(property "Intersheetrefs" "${INTERSHEET_REFS}"
-			(at 50.8 55.5995 90)
-			(effects
-				(font
-					(size 1.27 1.27)
-				)
-				(justify right)
-				(hide yes)
-			)
-		)
-	)
-	(global_label "+2v5exc"
+			(at 50.8 54.39 90)
+			(effects
+				(font
+					(size 1.27 1.27)
+				)
+				(justify right)
+				(hide yes)
+			)
+		)
+	)
+	(global_label "+5vexc"
 		(shape input)
 		(at 53.34 93.98 270)
@@
 		)
 		(property "Intersheetrefs" "${INTERSHEET_REFS}"
-			(at 53.34 105.1295 90)
-			(effects
-				(font
-					(size 1.27 1.27)
-				)
-				(justify right)
-				(hide yes)
-			)
-		)
-	)
-	(global_label "-2v5exc"
+			(at 53.34 103.92 90)
+			(effects
+				(font
+					(size 1.27 1.27)
+				)
+				(justify right)
+				(hide yes)
+			)
+		)
+	)
+	(global_label "-5vexc"
 		(shape input)
 		(at 53.34 78.74 90)
@@
 		)
 		(property "Intersheetrefs" "${INTERSHEET_REFS}"
-			(at 53.34 67.5905 90)
-			(effects
-				(font
+			(at 53.34 68.8 90)
+			(effects
+				(font
