File: 21xt/dyno_inst/voltages.kicad_sch (KiCad schematic)
At the start: 26 parts, among them IC1 TC7660SEOA713, U3 LM2587SX-12_NOPB, U4 LM4040A82IDBZT, U5 OPA2188AIDGKR, U6 ADR3425ARJZ-R7, U9 OPA2188AIDGKR

Commit message: ye
Parts:
- removed C11: 100u, symbol Device:C
- removed C12: 0.1u, symbol Device:C
- removed C13: 1u, symbol Device:C
- removed C20: 1uF, Capacitor_SMD:C_0402_1005Metric, symbol Device:C
- removed D1: D_Schottky, symbol Device:D_Schottky
- removed L1: 15uH, symbol Device:L
- removed PS1: AP2120N-2.5TRG1, SOT96P240X120-3N, symbol dyno_inst_sym:AP2120N-5.0TRG1
- removed R1: 3k, symbol Device:R
- removed R17, R9: 100k, symbol Device:R
- removed R2: 29.4, symbol Device:R
- removed U3: LM2587SX-12_NOPB, LM2587SX-12_NOPB:VREG_TPS79625KTTR, symbol dyno_inst_sym:LM2587SX-12_NOPB
- removed U4: LM4040A82IDBZT, DBZ3, symbol dyno_inst_sym:LM4040A82IDBZT
- removed U6: ADR3425ARJZ-R7, RJ_6_ADI, symbol dyno_inst_sym:ADR3425ARJZ-R7
- added C16: 0.1uf, Capacitor_SMD:C_0402_1005Metric, symbol Device:C
- added C17, C18: 10uF, Capacitor_SMD:C_0402_1005Metric, symbol Device:C
- added C22, C23: 0.01uf, Capacitor_SMD:C_0402_1005Metric, symbol Device:C
- added IC3: MCP1502T-25E_CHY, SOT95P280X145-6N, symbol dyno_inst_sym:MCP1502T-50E_CHY
- added J4: Barrel_Jack, symbol Connector:Barrel_Jack
- added U12: LT3032IDE-5-TRPBF, DFN14_DE14MA_ADI, symbol dyno_inst_sym:LT3032IDE-5-TRPBF
- added U13: REF3450QDBVRQ1, SOT-23-6_TEX, symbol dyno_inst_sym:REF3450QDBVRQ1
- added U6: 1S4E_1.5U, symbol dyno_inst_sym:1S4E_0505S1.5U
- C14: value 1200uF -> 0.1uf; footprint (none) -> Capacitor_SMD:C_0402_1005Metric
- C15: value 1200uF -> 1uF; footprint (none) -> Capacitor_SMD:C_0402_1005Metric
- C19: value 10uF -> 0.01uf
- C21: value 1uF -> 0.01uf
- renumbered C18 to C13, R3 to R18, R6 to R19, R8 to R20, R7 to R21, U9 to U7, U5 to U8
Connections:
- net +12v: now also C17.2, J4.1, U12.12 (*SHDNP), U12.14 (INP), U13.3 (ENABLE), U13.4 (IN), U6.2 (Vin); no longer C14.1, C15.1
- net -12v: now also C18.1, U12.16 (INN), U12.6 (INN), U12.9 (INN)
- net GNDA: now also C14.1, C15.1, C16.1, C17.1, C18.2, C22.1, C23.1, IC3.2 (GND_1), IC3.3 (GND_2), IC3.5 (GND_3), U12.10 (*SHDNN), U12.15 (GND), U12.4 (GND), U12.5 (GND), U13.1 (GND_F), U13.2 (GND_S); no longer C19.2, C21.2, U7.5 (INB+)
- net GNDPWR: now also U6.1 (GND); no longer C14.2, C15.2
- net +2v5exc renamed -5vexc
- net -5vexc: now also C23.2, U12.11 (BYPN)
- net +8v2ref renamed +5vref
- net +5vref: now also C14.2, C16.2, IC3.4 (~{SHDN}), IC3.6 (VDD), U13.5 (OUT_S), U13.6 (OUT_F)
- net -2v5exc: no longer names the net of U7.7 (OUTB)
- net -8v2ref renamed -5vref
- net 5v renamed +5vexc
- net +5vexc: now also C22.2, U12.1 (OUTP)
- new net: C21.2, U12.3 (BYPP)
- new net: C19.2, U12.7 (OUTN)
- new net +2v5vref: C15.2, IC3.1 (OUT)
- new net 5vpwr: U6.4 (+Vo)
- new net GND3: U6.3 (0V)
- no-connect marks 6 -> 8
Other:
- note added: "0.8/uS slew rate"
- note added: "find another op amp if needed. need: low supply in curr high psrr slew rate >= 0.1 V/us ish"
- note added: "separate excitation from sg b/c emi"
- note added: "stable 5v for creating negative ref v"
- note added: "teesny power, 5v isolated"
- note removed: "RR1220Q-29R4-D-M maybe"
- note removed: "for 8v2ref, -12v"
- note removed: "for inst amp ref, might as well try to max out fsr more stable than +/- 12v for creating negative exc v optiona imo, it is $3.86"
- note removed: "optimal"
- note removed: "separate excitation from sg b/c emi, ratiometric in sw i think better"
- note removed: "suboptimal lots of wasted current"
- moved on the sheet: C13, IC1, R18, R19, U7

Commit message: ye
Parts:
- added C32, C33: 10uF, Capacitor_SMD:C_0402_1005Metric, symbol Device:C
- added U15: R-78E5.0-0.5, R-78E-0.5_RCP, symbol dyno_inst_sym:R-78E5.0-0.5
Connections:
- net +12v: now also C32.1, U15.1 (+VIN)
- net GNDPWR: now also C32.2, C33.2, U15.2 (GND)
- new net 5venc: C33.1, U15.3 (+VOUT)
Other:
- moved on the sheet: C16, C17, C18, C19, C21, C22, C23, J4, R20, R21, U12, U13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

Commit message: sad
Parts:
- removed R18, R19, R20, R21: 100k, symbol Device:R
- removed U13: REF3450QDBVRQ1, SOT-23-6_TEX, symbol dyno_inst_sym:REF3450QDBVRQ1
- removed U7, U8: OPA2188AIDGKR, DGK8, symbol dyno_inst_sym:OPA2188AIDGKR
- added C35: 1uF, Capacitor_SMD:C_0402_1005Metric, symbol Device:C
- added C36: 0.1uf, Capacitor_SMD:C_0402_1005Metric, symbol Device:C
- added C37, C38, C39: 0.01uf, Capacitor_SMD:C_0402_1005Metric, symbol Device:C
- added C40, C41: 10uF, Capacitor_SMD:C_0402_1005Metric, symbol Device:C
- added IC2: MCP1502T-25E_CHY, SOT95P280X145-6N, symbol dyno_inst_sym:MCP1502T-50E_CHY
- added R5: 100k, symbol Device:R
- added U13: NCV8184DR2G, SOIC-8_NB_ONS, symbol dyno_inst_sym:NCV8184DR2G
- added U7: LT3032IDE-5-TRPBF, DFN14_DE14MA_ADI, symbol dyno_inst_sym:LT3032IDE-5-TRPBF
- C16: value 0.1uf -> 0.01uf
Connections:
- net +2v5vref is gone; now on net +2v5ref: C15.2, IC3.1 (OUT)
- net +12v: now also C41.2, U7.12 (*SHDNP), U7.14 (INP)
- net +2v5ref: now also R5.2
- net +5vref: now also C36.2, C37.1, IC2.4 (~{SHDN}), IC2.6 (VDD), U7.1 (OUTP)
- net -12v: now also C40.1, U7.16 (INN), U7.6 (INN), U7.9 (INN)
- net -5vref: now also C38.1, C39.2, U7.11 (BYPN)
- net GNDA: now also C35.1, C36.1, C39.1, C40.2, C41.1, IC2.2 (GND_1), IC2.3 (GND_2), IC2.5 (GND_3), U7.10 (*SHDNN), U7.15 (GND), U7.4 (GND), U7.5 (GND)
- new net: C37.2, U7.3 (BYPP)
- new net: C38.2, U7.7 (OUTN)
- new net +2v5adc: C35.2, IC2.1 (OUT)
- no-connect marks 8 -> 2
Other:
- note added: "+2v5ref -2v5ref 3v3 5venc"
- note added: "300 uA"
- note removed: "0.8/uS slew rate"
- note removed: "find another op amp if needed. need: low supply in curr high psrr slew rate >= 0.1 V/us ish"
- note removed: "for adc"
- note removed: "for dc transducer"
- note removed: "near optimal imo psrr is quite high"
- note removed: "separate excitation from sg b/c emi"
- note removed: "stable 5v for creating negative ref v"
- moved on the sheet: C14, C15, IC3, U6

Commit message: sche
Parts:
- added C29, C30, C33, C34: 0.1uf, Capacitor_SMD:C_0402_1005Metric, symbol Device:C
- added R10, R9: 100, symbol Device:R
- added R6: 500, symbol Device:R
- added R7, R8: 45k, symbol Device:R
- added U8, U9: TL431DBZ, Package_TO_SOT_SMD:SOT-23, symbol Reference_Voltage:TL431DBZ
- R5: value 100k -> 500
- U10: renamed from U12; footprint DFN14_DE14MA_ADI -> dynoinst_fp:DFN14_DE14MA_ADI
- U11: renamed from U13; footprint SOIC-8_NB_ONS -> dynoinst_fp:SOIC-8_NB_ONS
- U5: renamed from U7; footprint DFN14_DE14MA_ADI -> dynoinst_fp:DFN14_DE14MA_ADI
- U7: renamed from U15; footprint R-78E-0.5_RCP -> dynoinst_fp:R-78E-0.5_RCP
- renumbered C13 to C18, C16 to C19, C37 to C20, C38 to C21, C39 to C22, C15 to C23, C14 to C24, C32 to C25, C40 to C26, C41 to C27, C35 to C28, C33 to C31, C36 to C32, C22 to C35, C21 to C36, C19 to C37, C23 to C38, C18 to C39, C17 to C40, IC3 to IC1, IC1 to IC2, IC2 to IC3
Connections:
- net +2v5ref: no longer R5.2
- net -5vref: now also R5.1, R6.1
- net 5venc: now also U11.8 (VIN), C33.2
- net GNDA: now also C29.1, C30.1, R10.2, R9.2, U8.1 (K), U9.1 (K)
- net 3v3Ext: now reaches U11.1 (VOUT)
- net 3v3Ext: now also U11.4 (ADJ)
- net GND2: now reaches U11.2 (GND)
- net GND2: now also U11.3 (GND), U11.6 (GND), U11.7 (GND), C33.1
- net 3v3Teensy: now reaches U11.5 (VREF/ENABLE)
- net 3v3Teensy: now also C34.2
- new net: R7.2, R9.1, U8.2 (REF)
- new net: R10.1, R8.2, U9.2 (REF)
- new net -2v5adc: C29.2, R5.2, R7.1, U8.3 (A)
- new net -2v5ref: C30.2, R6.2, R8.1, U9.3 (A)
- new net GNDD: C34.1
Other:
- note added: "A C"
- note added: "coupled 3v3"
- note removed: "+2v5ref -2v5ref 3v3 5venc"
- moved on the sheet: C19, C20, C21, C22, C26, C27, U11, U5

Commit message: ye
Parts:
- C18: footprint (none) -> Capacitor_SMD:C_0603_1608Metric
- IC1, IC3: footprint SOT95P280X145-6N -> dynoinst_fp:SOT95P280X145-6N
- IC2: footprint SOIC127P600X175-8N -> dynoinst_fp:SOIC127P600X175-8N
- J4: footprint (none) -> dynoinst_fp:CUI_PJ-037A
- R10, R5, R6, R7, R8, R9: footprint (none) -> Resistor_SMD:R_0402_1005Metric
- U6: footprint (none) -> Connector_PinHeader_2.54mm:PinHeader_1x04_P2.54mm_Horizontal
Changed lines of the file:
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@@
 			)
 		)
-		(property "Footprint" ""
+		(property "Footprint" "Connector_PinHeader_2.54mm:PinHeader_1x04_P2.54mm_Horizontal"
 			(at 48.26 55.88 0)
 			(effects
@@
 			)
 		)
-		(property "Footprint" ""
+		(property "Footprint" "Resistor_SMD:R_0402_1005Metric"
 			(at 133.35 154.178 90)
 			(effects
@@
 			)
 		)
-		(property "Footprint" ""
+		(property "Footprint" "Resistor_SMD:R_0402_1005Metric"
 			(at 147.32 124.968 90)
 			(effects
@@
 			)
 		)
-		(property "Footprint" "SOT95P280X145-6N"
+		(property "Footprint" "dynoinst_fp:SOT95P280X145-6N"
 			(at 67.31 196.52 0)
 			(effects
@@
 			)
 		)
-		(property "Footprint" "SOIC127P600X175-8N"
+		(property "Footprint" "dynoinst_fp:SOIC127P600X175-8N"
 			(at 90.17 127.94 0)
 			(effects
@@
 			)
 		)
-		(property "Footprint" ""
+		(property "Footprint" "Resistor_SMD:R_0402_1005Metric"
 			(at 134.62 124.968 90)
 			(effects
@@
 			)
 		)
-		(property "Footprint" ""
+		(property "Footprint" "Capacitor_SMD:C_0603_1608Metric"
 			(at 33.9852 41.91 0)
 			(effects
@@
 			)
 		)
-		(property "Footprint" "SOT95P280X145-6N"
+		(property "Footprint" "dynoinst_fp:SOT95P280X145-6N"
 			(at 144.78 196.52 0)
 			(effects
@@
 			)
 		)
-		(property "Footprint" ""
+		(property "Footprint" "Resistor_SMD:R_0402_1005Metric"
 			(at 120.65 125.222 90)
 			(effects
@@
 			)
 		)
-		(property "Footprint" ""
+		(property "Footprint" "Resistor_SMD:R_0402_1005Metric"
 			(at 146.05 154.178 90)
 			(effects
@@
 			)
 		)
-		(property "Footprint" ""
+		(property "Footprint" "Resistor_SMD:R_0402_1005Metric"
 			(at 119.38 154.432 90)
 			(effects
@@
 			)
 		)
-		(property "Footprint" ""
+		(property "Footprint" "dynoinst_fp:CUI_PJ-037A"
 			(at 20.32 26.416 0)
 			(effects

Commit message: adasd
Other:
- note added: "+/-2v5 for FDA, adc ref"
- note added: "+/-2v5 for adc pwr"
- note added: "cruddy high current biplolar"
- note added: "encoder"
- note added: "filter ref+for +/-2v5 refs"
- note added: "in"
- note added: "sg excite"
- note removed: "?"
- note removed: "for negative power supply to create tracking +/-5v supply"
- note removed: "works"
- moved on the sheet: C18, C23, C24, C25, C28, C31, C32, C33, C34, C35, C36, C37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

Commit message: sss
Parts:
- added C69: 100uF, Capacitor_SMD:C_0805_2012Metric, symbol Device:C
- added C70: 10uF, Capacitor_SMD:C_0603_1608Metric, symbol Device:C
- C25, C31: footprint Capacitor_SMD:C_0402_1005Metric -> Capacitor_SMD:C_0603_1608Metric
- U6: footprint Connector_PinHeader_2.54mm:PinHeader_1x04_P2.54mm_Horizontal -> Connector_PinHeader_2.54mm:PinHeader_1x04_P2.54mm_Vertical
Connections:
- net +12v: now also C69.2, C70.2
- net GNDPWR: now also C69.1, C70.1

Commit message: stary layout
Parts:
- added C79, C80, C81, C82: 0.01uf, Capacitor_SMD:C_0402_1005Metric, symbol Device:C
- added C83, C84: 10uF, Capacitor_SMD:C_0402_1005Metric, symbol Device:C
- added U24: LT3032IDE-5-TRPBF, dynoinst_fp:DFN14_DE14MA_ADI, symbol dyno_inst_sym:LT3032IDE-5-TRPBF
Connections:
- net +12v: now also C84.2, U24.12 (*SHDNP), U24.14 (INP)
- net -12v: now also C83.1, U24.16 (INN), U24.6 (INN), U24.9 (INN)
- net GNDA: now also C79.1, C82.1, C83.2, C84.1, U24.10 (*SHDNN), U24.15 (GND), U24.4 (GND), U24.5 (GND)
- new net: C80.2, U24.3 (BYPP)
- new net: C81.2, U24.7 (OUTN)
- new net +5vcla: C79.2, C80.1, U24.1 (OUTP)
- new net -5vcla: C81.1, C82.2, U24.11 (BYPN)
