File: 21xt/dyno_inst/dyno_inst.kicad_pcb (KiCad board)
At the start: 4 copper layers, 151 parts, among them IC1 MCP1502T-25E_CHY, IC2 TC7660SEOA713, IC3 MCP1502T-25E_CHY, J4 Barrel_Jack, U1 MAX14931FASE+, U10 LT3032IDE-5-TRPBF, U11 NCV8184DR2G, U12 1SS362FV_L3F, U13 1SS362FV_L3F, U14 ADA4807-2ARM, U15 ADA4807-2ARM, U16 ADA4945-1ACPZ-R2, U17 1SS362FV_L3F, U18 1SS362FV_L3F, U19 ADA4807-1, U2 MAX14930FASE+, U20 ADA4807-1, U21 1SS362FV_L3F, U22 ADA4945-1ACPZ-R2, U23 CPC1017N, U3 AD7175-2BRUZ, U4 DEV-16771, U5 LT3032IDE-5-TRPBF, U6 1S4E_1.5U, U7 R-78E5.0-0.5, U8 TL431DBZ, U9 TL431DBZ

Commit message: layout start
Parts:
- moved J4 135.1 mm to (138.9, 93.9)
- moved C18 132.0 mm to (129.9, 72.4), turned to 180 degrees
- moved C25 126.0 mm to (142.5, 111.4)
- moved C31 126.0 mm to (156.8, 111.2)
- moved U7 126.0 mm to (147.1, 110.5)
- moved IC2 125.1 mm to (130.7, 77.2), turned to -90 degrees
- moved C19 124.4 mm to (143.3, 74.1), turned to 0 degrees
- moved C28 123.1 mm to (149.8, 73.0), turned to 90 degrees
- moved C20 122.8 mm to (143.3, 75.3), turned to 180 degrees
- moved C24 122.7 mm to (149.7, 80.2), turned to 90 degrees
- moved C70 121.7 mm to (134.3, 79.4), turned to -90 degrees
- moved IC3 120.5 mm to (147.3, 74.2), turned to -90 degrees
- moved IC1 120.2 mm to (147.2, 81.5), turned to -90 degrees
- moved C21 120.1 mm to (139.2, 77.1), turned to 90 degrees
- moved C32 119.7 mm to (149.8, 75.5), turned to -90 degrees
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Routing:
- net -2v5ref: track 0.00 -> 6.55 mm, vias 0 -> 4
- net +2v5ref: track 0.00 -> 6.50 mm, vias 0 -> 4
- net -intout: track 0.00 -> 4.16 mm
- net +DCSIG^': track 0.00 -> 4.16 mm
- net +intout: track 0.00 -> 4.12 mm
- net -DCSIG^': track 0.00 -> 4.07 mm
- net Net-(U16-+FB): track 0.00 -> 2.53 mm
- net Net-(U22-+FB): track 0.00 -> 2.48 mm
- net Net-(U22--FB): track 0.00 -> 2.46 mm
- net Net-(U16--FB): track 0.00 -> 2.46 mm
Other:
- board text added: ":("

Commit message: stary layout
Parts:
- added C79: 0.01uf, Capacitor_SMD:C_0402_1005Metric, F.Cu at (136.7, 91.5)
- added C80: 0.01uf, Capacitor_SMD:C_0402_1005Metric, F.Cu at (135.7, 91.5)
- added C81: 0.01uf, Capacitor_SMD:C_0402_1005Metric, F.Cu at (133.9, 87.5)
- added C82: 0.01uf, Capacitor_SMD:C_0402_1005Metric, F.Cu at (131.9, 87.5)
- added C83: 10uF, Capacitor_SMD:C_0402_1005Metric, F.Cu at (130.3, 88.9)
- added C84: 10uF, Capacitor_SMD:C_0402_1005Metric, F.Cu at (130.3, 91.9)
- added U24: LT3032IDE-5-TRPBF, dynoinst_fp:DFN14_DE14MA_ADI, F.Cu at (133.0, 90.5)
- moved C39 48.7 mm to (120.5, 89.1)
- moved C40 47.5 mm to (120.7, 92.1), turned to 90 degrees
- moved C38 44.9 mm to (122.4, 87.6), turned to 0 degrees
- moved U10 42.0 mm to (123.5, 90.6), turned to 180 degrees
- moved C37 41.0 mm to (124.3, 87.6), turned to 0 degrees
- moved C2 40.9 mm to (180.6, 109.0)
- moved C3 40.9 mm to (189.4, 109.1)
- moved U2 40.9 mm to (185.0, 114.0)
- moved C16 38.8 mm to (231.9, 66.3)
- moved R2 38.8 mm to (210.9, 94.8)
- moved R3 38.8 mm to (210.9, 99.8)
- moved U4 38.8 mm to (221.5, 96.0)
- moved R1 38.8 mm to (231.9, 99.8)
- moved R4 38.8 mm to (210.9, 97.3)
- moved C36 36.6 mm to (126.1, 91.6), turned to 90 degrees
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Connections:
- C37 pad 1: +DCEXC -> -5vexc
- C38 pad 2: +DCEXC -> -5vexc
- CR3 pad 2: +DCEXC -> +5vexc
- CR4 pad 2: +5vexc -> -5vexc
- U10 pad 11: +DCEXC -> -5vexc
- U12 pad 1: +DCEXC -> -5vcla
- U12 pad 2: +5vexc -> +5vcla
- U13 pad 1: +DCEXC -> -5vcla
- U13 pad 2: +5vexc -> +5vcla
- U17 pad 1: +DCEXC -> -5vcla
- U17 pad 2: +5vexc -> +5vcla
- U17 pad 3: +DCEXC -> +5vexc
- U18 pad 1: +DCEXC -> -5vcla
- U18 pad 2: +5vexc -> +5vcla
- U18 pad 3: +5vexc -> -5vexc
- U21 pad 1: +DCEXC -> -5vcla
- U21 pad 2: +5vexc -> +5vcla
- U3 pad 21: +DCSIG^'* -> -DCSIG^'*
- U3 pad 22: -DCSIG^'* -> +DCSIG^'*
Routing:
- net 5vpwr: track 0.00 -> 134.4 mm, vias 0 -> 1
- net +12v: track 0.00 -> 30.6 mm, vias 0 -> 6
- net +DCSIG^'*: track 0.00 -> 14.5 mm
- net -12v: track 0.00 -> 14.4 mm, vias 0 -> 6
- net -5vref: track 0.00 -> 14.1 mm
- net -DCSIG^'*: track 0.00 -> 13.4 mm
- net +5vref: track 0.00 -> 11.9 mm
- net +2v5ref: track 6.50 -> 14.5 mm
- net 5venc: track 0.00 -> 7.54 mm
- net 3v3Ext: track 0.00 -> 7.46 mm
- net Net-(C50-Pad1): track 0.00 -> 6.02 mm
- net Net-(C48-Pad1): track 0.00 -> 5.99 mm
- net Net-(U15B--): track 0.00 -> 5.60 mm
- net Net-(U15A--): track 0.00 -> 5.21 mm
- net +DCSIG^: track 0.00 -> 5.16 mm
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- added copper zone on In2.Cu, net +12v
- added copper zone on In2.Cu, net -12v
Other:
- board text removed: ":("

Commit message: ffff
Parts:
- added J1: Conn_01x05, Connector_PinHeader_2.54mm:PinHeader_1x05_P2.54mm_Vertical, F.Cu at (174.0, 125.0)
- added J5: Conn_01x06, Connector_PinHeader_2.54mm:PinHeader_1x06_P2.54mm_Vertical, F.Cu at (100.8, 104.8)
- added J6: Conn_01x04, peripheralio:CONN_T4041017041-000_TEC, F.Cu at (117.8, 72.6)
- moved R41 72.0 mm to (211.7, 62.2)
- moved U23 72.0 mm to (206.8, 60.9)
- moved C28 38.2 mm to (198.5, 70.2)
- moved C32 38.2 mm to (198.5, 72.7)
- moved IC3 38.2 mm to (196.0, 71.5)
- moved C29 35.3 mm to (200.0, 78.1)
- moved R5 35.3 mm to (201.5, 81.2)
- moved R7 35.3 mm to (199.9, 82.8)
- moved R9 35.3 mm to (196.3, 81.2)
- moved U8 35.3 mm to (199.0, 80.5)
- moved R6 28.9 mm to (150.6, 57.5)
- moved R10 28.9 mm to (145.3, 57.5)
- moved R8 28.9 mm to (149.0, 59.1)
- moved U9 28.9 mm to (148.0, 56.8)
- moved C30 28.9 mm to (149.0, 54.4)
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Connections:
- U4 pad 16: unconnected-(U4-A2-Pad16) -> BOTINB
- U4 pad 17: unconnected-(U4-A3-Pad17) -> TOPINB
- U4 pad 18: unconnected-(U4-A4-Pad18) -> BOTINA
- U4 pad 19: unconnected-(U4-A5-Pad19) -> TOPINA
Routing:
- net +5vexc: track 0.00 -> 24.4 mm
- net GNDA: track 0.00 -> 19.7 mm, vias 0 -> 15
- net -5vref: track 14.1 -> 26.9 mm
- net -5vcla: track 1.05 -> 13.5 mm
- net +5vref: track 11.9 -> 22.5 mm
- net -5vexc: track 1.05 -> 10.6 mm
- net GNDPWR: track 0.00 -> 7.24 mm, vias 0 -> 5
- net +5vcla: track 2.32 -> 9.11 mm
- net 5vpwr: track 134.4 -> 129.6 mm
- net -12v: track 14.4 -> 12.0 mm
- net Net-(U5-OUTN): track 0.00 -> 1.65 mm
- net Net-(U10-OUTN): track 0.00 -> 1.57 mm
- net Net-(U5-BYPP): track 0.00 -> 1.41 mm
- net Net-(U10-BYPP): track 0.00 -> 1.31 mm
- added copper zone on In1.Cu, net GNDA
- added copper zone on In1.Cu, net GNDPWR

Commit message: aaa
Parts:
- removed R39: 7.5, Resistor_SMD:R_0805_2012Metric
- removed U21: 1SS362FV_L3F, Package_TO_SOT_SMD:SOT-723
- added J3: Conn_01x03, peripheralio:CONN_T4041017041-000_TEC, F.Cu at (128.9, 81.1)
- moved J5 96.1 mm to (194.8, 124.5), turned to -90 degrees
- moved J1 68.3 mm to (204.9, 64.0)
- moved R1 54.6 mm to (179.5, 115.2), turned to 90 degrees
- moved C16 52.5 mm to (213.0, 115.2), turned to 180 degrees
- moved U23 49.8 mm to (166.6, 90.2)
- moved R41 49.8 mm to (171.4, 91.5)
- moved U4 39.2 mm to (183.3, 104.8), turned to 180 degrees
- moved R40 35.1 mm to (95.3, 78.2)
- moved CR5 35.1 mm to (98.1, 79.5)
- moved U2 32.8 mm to (202.3, 86.1), turned to 90 degrees
- moved R3 31.9 mm to (179.5, 94.2), turned to -90 degrees
- moved R4 29.0 mm to (182.0, 94.2), turned to -90 degrees
- moved C3 28.5 mm to (197.3, 81.6), turned to 0 degrees
- moved R2 26.4 mm to (184.5, 94.3), turned to -90 degrees
- moved C2 25.0 mm to (197.3, 90.5), turned to 0 degrees
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Connections:
- C2 pad 2: 5venc -> 3v3Teensy
- C3 pad 2: 3v3Teensy -> Net-(U2-VDDB)
- J6 pad 1: -DCSIG -> +5vexc
- J6 pad 2: +5vexc -> -DCSIG
- R40 pad 1: Net-(U21-C1/A2) -> ACSIG
- U1 pad 10: 3v3 -> 3v3Ext
- U1 pad 12: !BCS -> BMOSI
- U1 pad 13: BMOSI -> BSCLK
- U1 pad 14: BSCLK -> !BCS
- U1 pad 3: ASCLK -> !ACS
- U1 pad 4: AMOSI -> ASCLK
- U1 pad 5: !ACS -> AMOSI
- U1 pad 7: 3v3 -> 3v3Teensy
- U16 pad 16: GNDD -> GNDA
- U16 pad 17: GNDD -> GNDA
- U2 pad 1: 5venc -> 3v3Teensy
- U2 pad 10: 3v3 -> 5venc
- U2 pad 12: Benc3 -> Aenc3
- U2 pad 13: Benc2 -> Aenc2
- U2 pad 14: Benc1 -> Aenc1
- U2 pad 16: 3v3Teensy -> Net-(U2-VDDB)
- U2 pad 3: Aenc1 -> Benc1
- U2 pad 4: Aenc2 -> Benc2
- U2 pad 5: Aenc3 -> Benc3
- U22 pad 16: GNDD -> GNDA
- U22 pad 17: GNDD -> GNDA
Routing:
- net 5vpwr: track 129.6 -> 0.00 mm, vias 1 -> 0
- net GNDA: track 19.7 -> 83.8 mm, vias 15 -> 51
- net -5vexc: track 10.6 -> 29.2 mm
- net BSCLK: track 0.00 -> 16.7 mm
- net BMOSI: track 0.00 -> 14.9 mm
- net !BCS: track 0.00 -> 14.6 mm
- net BMISO: track 0.00 -> 14.6 mm
- net +5vref: track 22.5 -> 36.9 mm, vias 0 -> 1
- net -5vcla: track 13.5 -> 26.6 mm, vias 0 -> 6
- net +DCSIG: track 0.00 -> 9.63 mm
- net -DCSIG: track 0.00 -> 9.59 mm
- net -2v5ref: track 11.6 -> 19.7 mm
- net +5vcla: track 9.11 -> 16.4 mm, vias 0 -> 6
- net -2v5adc: track 0.00 -> 7.00 mm
- net GND1: track 0.00 -> 4.11 mm, vias 0 -> 4
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- added copper zone on In2.Cu, net +2v5ref
- added copper zone on In2.Cu, net +5vcla
- added copper zone on In2.Cu, net -2v5ref
- added copper zone on In2.Cu, net -5vcla
- added copper zone on In1.Cu, net GND1
- added copper zone on In1.Cu, net GNDD

Commit message: scuffedd
Parts:
- removed C25, C31: 10uF, Capacitor_SMD:C_0603_1608Metric
- added C85: 1uF, Capacitor_SMD:C_0402_1005Metric, F.Cu at (190.7, 71.5)
- added C86: 0.1uF, Capacitor_SMD:C_0402_1005Metric, F.Cu at (188.8, 71.5)
- added C87: 100uF, Capacitor_SMD:C_0805_2012Metric, F.Cu at (117.8, 107.2)
- U7: value R-78E5.0-0.5 -> 1S4E_1.5U; footprint dynoinst_fp:R-78E-0.5_RCP -> Connector_PinHeader_2.54mm:PinHeader_1x04_P2.54mm_Vertical
- moved CR5 33.2 mm to (131.1, 82.9)
- moved R40 33.2 mm to (128.2, 81.5)
- moved R41 30.1 mm to (142.9, 81.9), turned to -90 degrees
- moved U23 29.4 mm to (138.7, 81.2)
- moved U7 23.1 mm to (117.4, 111.3)
- moved R38 16.8 mm to (167.0, 64.3)
- moved R37 16.2 mm to (166.9, 81.7)
- moved C69 15.4 mm to (133.1, 101.4)
- moved C2 13.0 mm to (208.2, 83.4)
- moved C3 13.0 mm to (208.2, 74.6)
- moved U2 13.0 mm to (213.1, 79.0)
- moved J3 11.5 mm to (117.5, 81.9), turned to -90 degrees
- moved U6 9.86 mm to (139.3, 101.6)
- moved C28 8.14 mm to (200.7, 70.0)
- moved C32 8.14 mm to (200.7, 67.5)
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Connections:
- C1 pad 1: GND3 -> GNDA
- C15 pad 1: GNDD -> GNDA
- C17 pad 1: GNDD -> GNDA
- C2 pad 1: GND2 -> GNDA
- C3 pad 1: GNDD -> GND2
- C33 pad 1: GND2 -> GNDA
- C33 pad 2: 5venc -> 5vpwr
- C34 pad 1: GNDD -> GNDA
- C4 pad 1: GNDD -> GNDA
- C5 pad 2: GNDD -> GNDA
- C6 pad 2: GNDD -> GNDA
- J3 pad 1: ACSIG -> GND1
- J3 pad 2: GND1 -> ACSIG
- U1 pad 15: GNDD -> GNDA
- U1 pad 2: GND2 -> GNDA
- U1 pad 8: GND2 -> GNDA
- U1 pad 9: GNDD -> GNDA
- U11 pad 2: GND2 -> GNDA
- U11 pad 3: GND2 -> GNDA
- U11 pad 6: GND2 -> GNDA
- U11 pad 7: GND2 -> GNDA
- U11 pad 8: 5venc -> 5vpwr
- U2 pad 15: GNDD -> GND2
- U2 pad 2: GND2 -> GNDA
- U2 pad 8: GND2 -> GNDA
- U2 pad 9: GNDD -> GND2
- U23 pad 2: GND3 -> GNDA
- U3 pad 15: GNDD -> GNDA
- U3 pad 17: GNDD -> GNDA
- U4 pad 0: Benc1 -> Benc3
- U4 pad 2: unconnected-(U4-OUT2-Pad2) -> Benc1
- U4 pad 7: Benc3 -> unconnected-(U4-RX2-Pad7)
- U7 pad 1: +12v -> GNDPWR
- U7 pad 2: GNDPWR -> +12v
- U7 pad 3: 5venc -> GND2
Routing:
- net 5venc: track 7.54 -> 195.7 mm
- net 5vpwr: track 0.00 -> 102.2 mm, vias 0 -> 2
- net shcalctrl: track 0.00 -> 69.4 mm, vias 0 -> 1
- net ACSIG^: track 0.00 -> 61.3 mm
- net -5vref: track 25.8 -> 80.2 mm, vias 1 -> 8
- net +5vref: track 36.9 -> 84.3 mm, vias 1 -> 6
- net 3v3Ext: track 5.14 -> 44.2 mm, vias 0 -> 2
- net GNDA: track 83.8 -> 117.7 mm, vias 51 -> 70
- net ASCLK: track 0.00 -> 32.0 mm
- net ACSHCAL: track 0.00 -> 20.4 mm, vias 0 -> 1
- net +DCSIG^'*: track 14.5 -> 33.6 mm
- net Benc1: track 0.00 -> 18.1 mm
- net Benc2: track 0.00 -> 17.6 mm
- net Benc3: track 0.00 -> 17.1 mm
- net AMISO: track 0.00 -> 15.8 mm
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- added copper zone on In2.Cu, net +5vref
- added copper zone on In2.Cu, net -5vref
- added copper zone on In2.Cu, net 3v3Teensy
- added copper zone on In1.Cu, net GND2
- added copper zone on In1.Cu, net GND3
- removed copper zone on In1.Cu, net GNDD
Other:
- board outline added: 118.1 x 71.1 mm
- board text added: "star point: - analog, digital, pwr galv iso from: teensy digital, teensy pwr galv iso from: encoder, transducer"

Commit message: ssss
Parts:
- added C25: 0.1uF, Capacitor_SMD:C_0402_1005Metric, F.Cu at (195.9, 113.4)
- added C31: 0.1uF, Capacitor_SMD:C_0402_1005Metric, F.Cu at (194.7, 120.1)
- added CHA GND: Conn_01x02, TerminalBlock_4Ucon:TerminalBlock_4Ucon_1x02_P3.50mm_Horizontal, F.Cu at (125.9, 62.3)
- added J2: Conn_01x10, Connector_PinHeader_2.54mm:PinHeader_1x10_P2.54mm_Vertical, F.Cu at (154.1, 122.8)
- added J7: Conn_01x02, TerminalBlock_4Ucon:TerminalBlock_4Ucon_1x02_P3.50mm_Horizontal, F.Cu at (215.7, 68.0)
- added U25: MAX14930FASE+, dynoinst_fp:21-0041_S16&plus_1_MXM, F.Cu at (189.7, 115.7)
- ENC1 ENC2 ENC3 5v GND: renamed from J1
- moved C2 13.2 mm to (218.1, 74.6), turned to 180 degrees
- moved C3 12.6 mm to (217.1, 83.5)
- moved R2 3.34 mm to (187.1, 92.1)
- moved R3 3.34 mm to (182.1, 92.1)
- moved R4 3.34 mm to (184.6, 92.1)
- moved U4 3.34 mm to (185.8, 102.7)
- moved ENC1 ENC2 ENC3 5v GND 2.58 mm to (209.2, 59.2)
- moved J5 2.27 mm to (195.0, 122.8)
- moved R1 2.24 mm to (180.3, 113.2)
- moved C33 1.76 mm to (153.1, 92.3)
- moved U11 1.76 mm to (157.6, 90.7)
- moved C34 1.76 mm to (154.7, 87.1)
- turned U2 to -90 degrees
Connections:
- C1 pad 1: GNDA -> GND1
- C10 pad 1: GNDA -> GND1
- C11 pad 1: GNDA -> GND1
- C12 pad 2: GNDA -> GND1
- C13 pad 2: GNDA -> GND1
- C14 pad 1: GNDA -> GND1
- C15 pad 1: GNDA -> GND1
- C16 pad 1: GND3 -> GND1
- C17 pad 1: GNDA -> GND1
- C19 pad 1: GNDA -> GND1
- C2 pad 1: GNDA -> GND2
- C2 pad 2: 3v3Teensy -> 5venc
- C22 pad 1: GNDA -> GND1
- C23 pad 1: GNDA -> GND1
- C24 pad 1: GNDA -> GND1
- C26 pad 2: GNDA -> GND1
- C27 pad 1: GNDA -> GND1
- C28 pad 1: GNDA -> GND1
- C29 pad 1: GNDA -> GND1
- C3 pad 1: GND2 -> GND1
- C3 pad 2: Net-(U2-VDDB) -> 3v3Teensy
- C30 pad 1: GNDA -> GND1
- C32 pad 1: GNDA -> GND1
- C33 pad 1: GNDA -> GND1
- C34 pad 1: GNDA -> GND1
- C35 pad 1: GNDA -> GND1
- C38 pad 1: GNDA -> GND1
- C39 pad 2: GNDA -> GND1
- C4 pad 1: GNDA -> GND1
- C40 pad 1: GNDA -> GND1
- C41 pad 2: GNDA -> GND1
- C43 pad 2: GNDA -> GND1
- C45 pad 2: GNDA -> GND1
- C46 pad 2: GNDA -> GND1
- C47 pad 2: GNDA -> GND1
- C49 pad 2: GNDA -> GND1
- C5 pad 2: GNDA -> GND1
- C51 pad 1: GNDA -> GND1
- C52 pad 1: GNDA -> GND1
- C53 pad 2: GNDA -> GND1
- C55 pad 2: GNDA -> GND1
- C57 pad 2: GNDA -> GND1
- C58 pad 2: GNDA -> GND1
- C59 pad 2: GNDA -> GND1
- C6 pad 2: GNDA -> GND1
- C60 pad 2: GNDA -> GND1
- C61 pad 2: GNDA -> GND1
- C62 pad 2: GNDA -> GND1
- C63 pad 2: GNDA -> GND1
- C64 pad 2: GNDA -> GND1
- C65 pad 2: GNDA -> GND1
- C66 pad 2: GNDA -> GND1
- C67 pad 1: GNDA -> GND1
- C68 pad 1: GNDA -> GND1
- C69 pad 1: GNDPWR -> GND1
- C7 pad 1: GNDA -> GND1
- C70 pad 1: GNDPWR -> GND1
- C71 pad 2: GNDA -> GND1
- C72 pad 2: GNDA -> GND1
- C73 pad 2: GNDA -> GND1
- C74 pad 2: GNDA -> GND1
- C75 pad 2: GNDA -> GND1
- C76 pad 2: GNDA -> GND1
- C77 pad 2: GNDA -> GND1
- C78 pad 2: GNDA -> GND1
- C79 pad 1: GNDA -> GND1
- C8 pad 1: GNDA -> GND1
- C82 pad 1: GNDA -> GND1
- C83 pad 2: GNDA -> GND1
- C84 pad 1: GNDA -> GND1
- C85 pad 1: GNDA -> GND1
- C86 pad 1: GNDA -> GND1
- C87 pad 1: GNDPWR -> GND1
- C9 pad 1: GNDA -> GND1
- IC1 pad 2: GNDA -> GND1
- IC1 pad 3: GNDA -> GND1
- IC1 pad 5: GNDA -> GND1
- IC2 pad 3: GNDPWR -> GND1
- IC3 pad 2: GNDA -> GND1
- IC3 pad 3: GNDA -> GND1
- IC3 pad 5: GNDA -> GND1
- J4 pad 2: unconnected-(J4-Pad2) -> GND1
- J5 pad 1: TOPINA -> TOPINA5v
- J5 pad 2: BOTINA -> BOTINA5v
- J5 pad 3: TOPINB -> TOPINB5v
- J5 pad 4: BOTINB -> BOTINB5v
- J5 pad 5: 5vpwr -> +12v
- J5 pad 6: GND3 -> GND1
- R10 pad 2: GNDA -> GND1
- R16 pad 1: GNDA -> GND1
- R17 pad 1: GNDA -> GND1
- R9 pad 2: GNDA -> GND1
- U1 pad 15: GNDA -> GND1
- U1 pad 2: GNDA -> GND1
- U1 pad 8: GNDA -> GND1
- U1 pad 9: GNDA -> GND1
- U10 pad 10: GNDA -> GND1
- U10 pad 15: GNDA -> GND1
- U10 pad 4: GNDA -> GND1
- U10 pad 5: GNDA -> GND1
- U11 pad 2: GNDA -> GND1
- U11 pad 3: GNDA -> GND1
- U11 pad 6: GNDA -> GND1
- U11 pad 7: GNDA -> GND1
- U16 pad 16: GNDA -> GND1
- U16 pad 17: GNDA -> GND1
- U16 pad 9: GNDA -> GND1
- U2 pad 1: 3v3Teensy -> 5venc
- U2 pad 10: 5venc -> 3v3Teensy
- U2 pad 12: Aenc3 -> Benc1
- U2 pad 13: Aenc2 -> Benc2
- U2 pad 14: Aenc1 -> Benc3
- U2 pad 15: GND2 -> GND1
- U2 pad 16: Net-(U2-VDDB) -> 3v3Teensy
- U2 pad 2: GNDA -> GND2
- U2 pad 3: Benc1 -> Aenc3
- U2 pad 4: Benc2 -> Aenc2
- U2 pad 5: Benc3 -> Aenc1
- U2 pad 8: GNDA -> GND2
- U2 pad 9: GND2 -> GND1
- U22 pad 16: GNDA -> GND1
- U22 pad 17: GNDA -> GND1
- U22 pad 9: GNDA -> GND1
- U23 pad 2: GNDA -> GND1
- U24 pad 10: GNDA -> GND1
- U24 pad 15: GNDA -> GND1
- U24 pad 4: GNDA -> GND1
- U24 pad 5: GNDA -> GND1
- U3 pad 15: GNDA -> GND1
- U3 pad 17: GNDA -> GND1
- U4 pad 14: unconnected-(U4-A0-Pad14) -> BOTINB3v3
- U4 pad 15: unconnected-(U4-A1-Pad15) -> TOPINB3v3
- U4 pad 16: BOTINB -> unconnected-(U4-A2-Pad16)
- U4 pad 17: TOPINB -> unconnected-(U4-A3-Pad17)
- U4 pad 18: BOTINA -> BOTINA3v3
- U4 pad 19: TOPINA -> TOPINA3v3
- U4 pad 34: unconnected-(U4-RX8-Pad34) -> INA
- U4 pad 35: unconnected-(U4-TX8-Pad35) -> ENA
- U4 pad 36: unconnected-(U4-CS2-Pad36) -> PWM
- U4 pad 37: unconnected-(U4-CS3-Pad37) -> CURRSNS
- U4 pad 38: unconnected-(U4-A14-Pad38) -> ENB
- U4 pad 39: unconnected-(U4-A15-Pad39) -> INB
- U5 pad 10: GNDA -> GND1
- U5 pad 15: GNDA -> GND1
- U5 pad 4: GNDA -> GND1
- U5 pad 5: GNDA -> GND1
- U6 pad 1: GNDPWR -> GND1
- U6 pad 3: GND3 -> GND1
- U7 pad 1: GNDPWR -> GND1
- U8 pad 1: GNDA -> GND1
- U9 pad 1: GNDA -> GND1
Routing:
- net GND1: track 6.45 -> 137.8 mm, vias 6 -> 86
- net GNDA: track 117.7 -> 0.00 mm, vias 70 -> 0
- net +12v: track 39.9 -> 75.1 mm
- net 3v3Teensy: track 10.3 -> 39.2 mm, vias 4 -> 6
- net 5vpwr: track 102.2 -> 125.8 mm, vias 2 -> 4
- net INB: track 0.00 -> 14.6 mm
- net INA: track 0.00 -> 14.6 mm
- net ENB: track 0.00 -> 14.6 mm
- net ENA: track 0.00 -> 14.6 mm
- net CURRSNS: track 0.00 -> 14.6 mm
- net PWM: track 0.00 -> 14.6 mm
- net TOPINA3v3: track 0.00 -> 6.81 mm
- net GNDPWR: track 6.73 -> 0.00 mm, vias 4 -> 0
- net TOPINA5v: track 0.00 -> 5.83 mm
- net BOTINA3v3: track 0.00 -> 5.50 mm
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- removed copper zone on In1.Cu, net GND3
- removed copper zone on In1.Cu, net GNDA
- removed copper zone on In1.Cu, net GNDPWR
Other:
- board text added: "+5vexc"
- board text added: "+DCSIG"
- board text added: "-5vexc"
- board text added: "-DCSIG"
- board text added: "0 Ohm DNP"
- board text added: "12v in"
- board text added: "ACSHCAL"
- board text added: "ACSIG"
- board text added: "BJR@JHU 21xt/dyno dyno inst"
- board text added: "CHA GND"
- board text added: "GND"
- board text added: "GND 12v BINB TINB BINA TINA"
- board text added: "INA ENA PWM CS ENB INB 5v GND NC GND"
- board text added: "NC"
- board text added: "U23"
- board text added: "big hbridge"
- board text added: "small hbridge"
- board text removed: "star point: - analog, digital, pwr galv iso from: teensy digital, teensy pwr galv iso from: encoder, transducer"
