File: 21xt/dyno_inst/dyno_inst.kicad_pcb (KiCad board)
At the start: 4 copper layers, 118.1 x 71.1 mm, 167 parts, among them IC1 MCP1502T-25E_CHY, IC2 TC7660SEOA713, IC3 MCP1502T-25E_CHY, J2 Conn_01x10, J3 Conn_01x03, J4 Barrel_Jack, J5 Conn_01x06, J6 Conn_01x04, J7 Conn_01x02, U1 MAX14931FASE+, U10 LT3032IDE-5-TRPBF, U11 NCV8184DR2G, U12 1SS362FV_L3F, U13 1SS362FV_L3F, U14 ADA4807-2ARM, U15 ADA4807-2ARM, U16 ADA4945-1ACPZ-R2, U17 1SS362FV_L3F, U18 1SS362FV_L3F, U19 ADA4807-1, U2 MAX14930FASE+, U20 ADA4807-1, U22 ADA4945-1ACPZ-R2, U23 CPC1017N, U24 LT3032IDE-5-TRPBF, U25 MAX14930FASE+, U3 AD7175-2BRUZ, U4 DEV-16771, U5 LT3032IDE-5-TRPBF, U6 1S4E_1.5U, U7 1S4E_1.5U, U8 TL431DBZ, U9 TL431DBZ

Commit message: aaaaa
Parts:
- removed C34: 0.1uf, Capacitor_SMD:C_0402_1005Metric
- removed CHA GND: Conn_01x02, TerminalBlock_4Ucon:TerminalBlock_4Ucon_1x02_P3.50mm_Horizontal
- removed U25: MAX14930FASE+, dynoinst_fp:21-0041_S16&plus_1_MXM
- added C91: 0.1uF, Capacitor_SMD:C_0402_1005Metric, F.Cu at (40.4, 10.6)
- added C92: 0.1uF, Capacitor_SMD:C_0402_1005Metric, F.Cu at (41.5, 10.6)
- added C93: 0.1uF, Capacitor_SMD:C_0402_1005Metric, F.Cu at (46.7, 10.6)
- added C94: 0.1uF, Capacitor_SMD:C_0402_1005Metric, F.Cu at (47.9, 10.6)
- added H1: MountingHole_Pad, MountingHole:MountingHole_3mm_Pad, F.Cu at (19.3, 43.2)
- added H2: MountingHole_Pad, MountingHole:MountingHole_3mm_Pad, F.Cu at (27.6, 89.2)
- added H3: MountingHole_Pad, MountingHole:MountingHole_3mm_Pad, F.Cu at (10.6, 43.2)
- added H4: MountingHole_Pad, MountingHole:MountingHole_3mm_Pad, F.Cu at (15.8, 0.30)
- added H5: MountingHole_Pad, MountingHole:MountingHole_3mm_Pad, F.Cu at (102.1, 1.80)
- added H6: MountingHole_Pad, MountingHole:MountingHole_3mm_Pad, F.Cu at (0.00, 0.00)
- added L1: 10uH, Inductor_SMD:L_1210_3225Metric, F.Cu at (88.7, 43.9)
- added R39: 100, Resistor_SMD:R_0402_1005Metric, F.Cu at (91.1, 42.1)
- added R45: 52.5, Resistor_SMD:R_0402_1005Metric, F.Cu at (40.4, -3.75)
- added R46: 52.5, Resistor_SMD:R_0402_1005Metric, F.Cu at (46.8, -3.70)
- added T1: 749013011, 21xt_footprints:749013011, F.Cu at (44.1, 3.21)
- added U21: CME0303S3C, dynoinst_fp:SIP4_CME0303_MUR, F.Cu at (81.8, 36.3)
- C33: value 0.1uf -> 4.7uF
- J1: renamed from ENC1 ENC2 ENC3 5v GND
- J7: value Conn_01x02 -> Conn_01x04; footprint TerminalBlock_4Ucon:TerminalBlock_4Ucon_1x02_P3.50mm_Horizontal -> peripheralio:CONN_T4041017041-000_TEC
- R1, R2, R3, R4: value tbd -> 20
- U11: value NCV8184DR2G -> MAX14930FASE+; footprint dynoinst_fp:SOIC-8_NB_ONS -> dynoinst_fp:21-0041_S16&plus_1_MXM
- moved J1 206.7 mm to (4.16, 33.2), turned to 180 degrees
- moved C3 206.3 mm to (19.6, 24.3), turned to -90 degrees
- moved C16 205.9 mm to (35.0, 11.8), turned to 0 degrees
- moved J7 197.5 mm to (31.3, -2.65)
- moved J5 185.4 mm to (54.5, 1.88), turned to 90 degrees
- moved C25 175.2 mm to (53.6, 11.3), turned to 0 degrees
- moved U2 168.6 mm to (59.8, 9.02), turned to 90 degrees
- moved C1 165.2 mm to (28.4, 25.2), turned to 90 degrees
- moved R1 150.7 mm to (69.1, 11.5), turned to -90 degrees
- moved U11 147.1 mm to (23.9, 29.2), turned to 0 degrees
- moved C4 146.9 mm to (54.7, 4.60)
- moved U4 146.5 mm to (63.6, 22.0), turned to 0 degrees
- moved C2 145.1 mm to (78.3, 35.8)
- moved C31 138.8 mm to (78.2, 44.8)
- moved R2 138.1 mm to (62.4, 32.7), turned to -90 degrees
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Connections:
- C1 pad 1: GND1 -> GND3
- C10 pad 1: GND1 -> GNDA
- C11 pad 1: GND1 -> GNDA
- C12 pad 2: GND1 -> GNDA
- C13 pad 2: GND1 -> GNDA
- C14 pad 1: GND1 -> GNDA
- C15 pad 1: GND1 -> GNDD
- C16 pad 1: GND1 -> GND3
- C17 pad 1: GND1 -> GNDD
- C19 pad 1: GND1 -> GNDA
- C2 pad 1: GND2 -> GND3
- C2 pad 2: 5venc -> 3v3Teensy
- C22 pad 1: GND1 -> GNDA
- C23 pad 1: GND1 -> GNDA
- C24 pad 1: GND1 -> GNDA
- C25 pad 1: GND1 -> GND3
- C26 pad 2: GND1 -> GNDA
- C27 pad 1: GND1 -> GNDA
- C28 pad 1: GND1 -> GNDA
- C29 pad 1: GND1 -> GNDA
- C3 pad 1: GND1 -> GND2
- C3 pad 2: 3v3Teensy -> 5venc
- C30 pad 1: GND1 -> GNDA
- C31 pad 1: GND1 -> GNDD
- C31 pad 2: 5vpwr -> 3v3Ext
- C32 pad 1: GND1 -> GNDA
- C33 pad 1: GND1 -> 3v3Ext
- C33 pad 2: 5vpwr -> GNDD
- C35 pad 1: GND1 -> GNDA
- C38 pad 1: GND1 -> GNDA
- C39 pad 2: GND1 -> GNDA
- C4 pad 1: GND1 -> GND3
- C4 pad 2: 3v3Ext -> 5vpwr
- C40 pad 1: GND1 -> GNDA
- C41 pad 2: GND1 -> GNDA
- C43 pad 2: GND1 -> GNDA
- C45 pad 2: GND1 -> GNDA
- C46 pad 2: GND1 -> GNDA
- C47 pad 2: GND1 -> GNDA
- C49 pad 2: GND1 -> GNDA
- C5 pad 2: GND1 -> GNDD
- C51 pad 1: GND1 -> GNDA
- C52 pad 1: GND1 -> GNDA
- C53 pad 2: GND1 -> GNDA
- C55 pad 2: GND1 -> GNDA
- C57 pad 2: GND1 -> GNDA
- C58 pad 2: GND1 -> GNDA
- C59 pad 2: GND1 -> GNDA
- C6 pad 2: GND1 -> GNDD
- C60 pad 2: GND1 -> GNDA
- C61 pad 2: GND1 -> GNDA
- C62 pad 2: GND1 -> GNDA
- C63 pad 2: GND1 -> GNDA
- C64 pad 2: GND1 -> GNDA
- C65 pad 2: GND1 -> GNDA
- C66 pad 2: GND1 -> GNDA
- C67 pad 1: GND1 -> GNDA
- C68 pad 1: GND1 -> GNDA
- C69 pad 1: GND1 -> GNDPWR
- C7 pad 1: GND1 -> GNDA
- C70 pad 1: GND1 -> GNDPWR
- C71 pad 2: GND1 -> GNDA
- C72 pad 2: GND1 -> GNDA
- C73 pad 2: GND1 -> GNDA
- C74 pad 2: GND1 -> GNDA
- C75 pad 2: GND1 -> GNDA
- C76 pad 2: GND1 -> GNDA
- C77 pad 2: GND1 -> GNDA
- C78 pad 2: GND1 -> GNDA
- C79 pad 1: GND1 -> GNDA
- C8 pad 1: GND1 -> GNDA
- C82 pad 1: GND1 -> GNDA
- C83 pad 2: GND1 -> GNDA
- C84 pad 1: GND1 -> GNDA
- C85 pad 1: GND1 -> GNDA
- C86 pad 1: GND1 -> GNDA
- C87 pad 1: GND1 -> GNDPWR
- C9 pad 1: GND1 -> GNDA
- IC1 pad 2: GND1 -> GNDA
- IC1 pad 3: GND1 -> GNDA
- IC1 pad 5: GND1 -> GNDA
- IC2 pad 3: GND1 -> GNDPWR
- IC3 pad 2: GND1 -> GNDA
- IC3 pad 3: GND1 -> GNDA
- IC3 pad 5: GND1 -> GNDA
- J2 pad 10: GND1 -> GND3
- J2 pad 8: GND1 -> GND3
- J4 pad 2: GND1 -> GNDPWR
- J5 pad 5: +12v -> 5vpwr
- J5 pad 6: GND1 -> GND3
- J7 pad 1: GND2 -> Rx+
- J7 pad 2: GND2 -> Rx-
- R10 pad 2: GND1 -> GNDA
- R16 pad 1: GND1 -> GNDA
- R17 pad 1: GND1 -> GNDA
- R9 pad 2: GND1 -> GNDA
- U1 pad 15: GND1 -> GNDD
- U1 pad 2: GND1 -> GND3
- U1 pad 8: GND1 -> GND3
- U1 pad 9: GND1 -> GNDD
- U10 pad 10: GND1 -> GNDA
- U10 pad 15: GND1 -> GNDA
- U10 pad 4: GND1 -> GNDA
- U10 pad 5: GND1 -> GNDA
- U11 pad 1: 3v3Ext -> 5venc
- U11 pad 2: GND1 -> GND2
- U11 pad 3: GND1 -> Aenc3
- U11 pad 4: 3v3Ext -> Aenc2
- U11 pad 5: 3v3Teensy -> Aenc1
- U11 pad 6: GND1 -> unconnected-(U11-INA4-Pad6)
- U11 pad 7: GND1 -> unconnected-(U11-I.C.-Pad7)
- U11 pad 8: 5vpwr -> GND2
- U16 pad 16: GND1 -> GNDA
- U16 pad 17: GND1 -> GNDA
- U16 pad 9: GND1 -> GNDA
- U2 pad 1: 5venc -> 3v3Teensy
- U2 pad 10: 3v3Teensy -> 5vpwr
- U2 pad 11: unconnected-(U2-OUTB4-Pad11) -> BOTINB5v
- U2 pad 12: Benc1 -> TOPINB5v
- U2 pad 13: Benc2 -> BOTINA5v
- U2 pad 14: Benc3 -> TOPINA5v
- U2 pad 15: GND1 -> GND3
- U2 pad 16: 3v3Teensy -> 5vpwr
- U2 pad 2: GND2 -> GND3
- U2 pad 3: Aenc3 -> TOPINA3v3
- U2 pad 4: Aenc2 -> BOTINA3v3
- U2 pad 5: Aenc1 -> TOPINB3v3
- U2 pad 6: unconnected-(U2-INA4-Pad6) -> BOTINB3v3
- U2 pad 8: GND2 -> GND3
- U2 pad 9: GND1 -> GND3
- U22 pad 16: GND1 -> GNDA
- U22 pad 17: GND1 -> GNDA
- U22 pad 9: GND1 -> GNDA
- U23 pad 2: GND1 -> GND3
- U24 pad 10: GND1 -> GNDA
- U24 pad 15: GND1 -> GNDA
- U24 pad 4: GND1 -> GNDA
- U24 pad 5: GND1 -> GNDA
- U3 pad 15: GND1 -> GNDD
- U3 pad 17: GND1 -> GNDD
- U4 pad GND1: unconnected-(U4-GND-PadGND1) -> GND3
- U4 pad GND2: unconnected-(U4-GND__1-PadGND2) -> GND3
- U4 pad GND3: unconnected-(U4-GND__2-PadGND3) -> GND3
- U4 pad GND4: unconnected-(U4-GND__3-PadGND4) -> GND3
- U4 pad GND5: unconnected-(U4-GND__4-PadGND5) -> GND3
- U4 pad R+: unconnected-(U4-PadR+) -> Rd+
- U4 pad R-: unconnected-(U4-PadR-) -> Rd-
- U4 pad T+: unconnected-(U4-PadT+) -> Td+
- U4 pad T-: unconnected-(U4-PadT-) -> Td-
- U4 pad USB_GND1: unconnected-(U4-USB_GND-PadUSB_GND1) -> GND3
- U4 pad USB_GND2: unconnected-(U4-USB_GND__1-PadUSB_GND2) -> GND3
- U5 pad 10: GND1 -> GNDA
- U5 pad 15: GND1 -> GNDA
- U5 pad 4: GND1 -> GNDA
- U5 pad 5: GND1 -> GNDA
- U6 pad 1: GND1 -> GNDPWR
- U6 pad 3: GND1 -> GND3
- U7 pad 1: GND1 -> GNDPWR
- U8 pad 1: GND1 -> GNDA
- U9 pad 1: GND1 -> GNDA
Routing:
- net GND1: track 137.8 -> 6.63 mm, vias 86 -> 6
- net GNDA: track 0.00 -> 106.5 mm, vias 0 -> 47
- net 5venc: track 197.7 -> 96.9 mm
- net 5vpwr: track 125.8 -> 219.0 mm, vias 4 -> 2
- net 3v3Teensy: track 39.2 -> 112.8 mm, vias 6 -> 4
- net -2v5ref: track 25.2 -> 63.0 mm, vias 9 -> 10
- net shcalctrl: track 68.3 -> 30.8 mm, vias 1 -> 0
- net +2v5ref: track 22.1 -> 59.5 mm, vias 8 -> 9
- net -5vref: track 80.4 -> 55.6 mm, vias 8 -> 7
- net +12v: track 75.1 -> 50.3 mm, vias 4 -> 6
- net +5vref: track 84.3 -> 59.9 mm
- net Tx+: track 0.00 -> 22.6 mm
- net Tx-: track 0.00 -> 22.6 mm
- net GND3: track 0.00 -> 21.9 mm, vias 0 -> 17
- net Td-: track 0.00 -> 19.0 mm
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- added copper zone on F.Cu, net -12v
- added copper zone on In1.Cu, net GND3
- added copper zone on In1.Cu, net GNDA
- added copper zone on In1.Cu, net GNDD
- added copper zone on In1.Cu, net GNDPWR
- removed copper zone on In2.Cu, net 3v3Teensy
Other:
- board size 118.1 x 71.1 mm -> 112.3 x 106.8 mm
- board text removed: "U23"

Commit message: adasd
Routing:
- net 3v3Teensy: track 112.8 -> 109.8 mm
- net 5vpwr: track 219.0 -> 219.9 mm
Other:
- board text added: "Rx+"
- board text added: "Rx-"
- board text added: "Tx+"
- board text added: "Tx-"
Changed lines of the file:
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@@
 		(tags "capacitor")
 		(property "Reference" "C2"
-			(at 0 -1.16 360)
+			(at 0 -1.16 0)
 			(layer "F.SilkS")
 			(effects
@@
 		)
 		(property "Value" "0.1uF"
-			(at 0 1.16 360)
+			(at 0 1.16 0)
 			(layer "F.Fab")
 			(effects
@@
 		)
 		(fp_text user "${REFERENCE}"
-			(at 0 0 360)
+			(at 0 0 0)
 			(layer "F.Fab")
 			(effects
@@
 		(tags "capacitor")
 		(property "Reference" "C31"
-			(at 0 -1.16 360)
+			(at 0 -1.16 0)
 			(layer "F.SilkS")
 			(effects
@@
 		)
 		(property "Value" "0.1uF"
-			(at 0 1.16 360)
+			(at 0 1.16 0)
 			(layer "F.Fab")
 			(effects
@@
 		)
 		(fp_text user "${REFERENCE}"
-			(at 0 0 360)
+			(at 0 0 0)
 			(layer "F.Fab")
 			(effects
@@
 		(tags "resistor")
 		(property "Reference" "R46"
-			(at 0 -1.17 360)
+			(at 0 -1.17 0)
 			(layer "F.SilkS")
 			(effects
@@
 		)
 		(property "Value" "52.5"
-			(at 0.11 0.975 360)
+			(at 0.11 0.975 0)
 			(layer "F.Fab")
 			(effects
@@
 		)
 		(fp_text user "${REFERENCE}"
-			(at 0 0 360)
+			(at 0 0 0)
 			(layer "F.Fab")
 			(effects
@@
 		(tags "resistor")
 		(property "Reference" "R41"
-			(at 0 -1.17 360)
+			(at 0 -1.17 0)
 			(layer "F.SilkS")
 			(effects
@@
 		)
 		(property "Value" "330"
-			(at 0 1.17 360)
+			(at 0 1.17 0)
 			(layer "F.Fab")
 			(effects
@@
 		)
 		(fp_text user "${REFERENCE}"
-			(at 0 0 360)
+			(at 0 0 0)
 			(layer "F.Fab")
 			(effects
@@
 		(tags "resistor")
 		(property "Reference" "R45"
-			(at 0 -1.17 360)
+			(at 0 -1.17 0)
 			(layer "F.SilkS")
 			(effects
@@
 		)
 		(property "Value" "52.5"
-			(at 0 1.17 360)
+			(at 0 1.17 0)
 			(layer "F.Fab")
 			(effects
@@
 		)
 		(fp_text user "${REFERENCE}"
-			(at 0 0 360)
+			(at 0 0 0)
 			(layer "F.Fab")
 			(effects
@@
 		(tags "capacitor")
 		(property "Reference" "C4"
-			(at 0 -1.16 360)
+			(at 0 -1.16 0)
 			(layer "F.SilkS")
 			(effects
@@
 		)
 		(property "Value" "0.1uF"
-			(at 0 1.16 360)
+			(at 0 1.16 0)
 			(layer "F.Fab")
 			(effects
@@
 		)
 		(fp_text user "${REFERENCE}"
-			(at 0 0 360)
+			(at 0 0 0)
 			(layer "F.Fab")
 			(effects
@@
 	)
 	(gr_circle
+		(center 30.325 6.964421)
+		(end 34.839421 6.964421)
+		(stroke
+			(width 0.1)
+			(type default)
+		)
+		(fill none)
+		(layer "B.SilkS")
+	)
+	(gr_circle
 		(center 16.67 50.889421)
 		(end 21.184421 50.889421)
@@
 		(layer "Edge.Cuts")
 	)
+	(gr_text "Rx-"
+		(at 33.15 4.925 0)
+		(layer "B.SilkS")
+		(effects
+			(font
+				(size 1 1)
+				(thickness 0.1)
+			)
+			(justify left bottom mirror)
+		)
+	)
 	(gr_text "ACSHCAL"
 		(at 19.795 58.6 0)
@@
 		)
 	)
+	(gr_text "Tx-"
+		(at 29.875 4.9 0)
+		(layer "B.SilkS")
+		(effects
+			(font
+				(size 1 1)
+				(thickness 0.1)
+			)
+			(justify left bottom mirror)
+		)
+	)
+	(gr_text "Rx+"
+		(at 34.25 7.25 0)
+		(layer "B.SilkS")
+		(effects
+			(font
+				(size 1 1)
+				(thickness 0.1)
+			)
+			(justify left bottom mirror)
+		)
+	)
 	(gr_text "-DCSIG"
 		(at 21.209421 50.689421 0)
@@
 		)
 	)
+	(gr_text "Tx+"
+		(at 29.1 7.375 0)
+		(layer "B.SilkS")
+		(effects
+			(font
+				(size 1 1)
+				(thickness 0.1)
+			)
+			(justify left bottom mirror)
+		)
+	)
 	(gr_text "NC"
 		(at 20.545 60.25 0)
@@
 	)
 	(gr_text "big hbridge"
-		(at 38.86 2.48 0)
+		(at 53.85 -2.425 0)
 		(layer "F.SilkS")
 		(effects
@@
 	)
 	(gr_text "small hbridge"
-		(at 76.96 5.757028 0)
+		(at 75.675 -1.75 0)
 		(layer "F.SilkS")
 		(effects
@@
 	)
 	(segment
-		(start 35.702721 18.547028)
-		(end 35.702721 13.447028)
+		(start 39.35 18.45)
+		(end 43.45 18.45)
 		(width 0.5)
 		(layer "In2.Cu")
@@
 	)
 	(segment
-		(start 50.349749 12.25)
-		(end 52.572721 10.027028)
+		(start 34.799749 19.45)
+		(end 38.35 19.45)
 		(width 0.5)
 		(layer "In2.Cu")
@@
 	)
 	(segment
-		(start 36.899749 12.25)
-		(end 50.349749 12.25)
+		(start 70.022721 35.702028)
+		(end 70.322721 35.402028)
 		(width 0.5)
 		(layer "In2.Cu")
@@
 	)
 	(segment
-		(start 70.022721 35.702028)
-		(end 70.322721 35.402028)
+		(start 29.447721 24.802028)
+		(end 34.799749 19.45)
 		(width 0.5)
 		(layer "In2.Cu")
@@
 	)
 	(segment
-		(start 35.702721 13.447028)
-		(end 36.899749 12.25)
+		(start 51.872972 10.027028)
+		(end 52.572721 10.027028)
+		(width 0.5)
+		(layer "In2.Cu")
+		(net 1)
+	)
+	(segment
+		(start 43.45 18.45)
+		(end 51.872972 10.027028)
 		(width 0.5)
 		(layer "In2.Cu")
@@
 	)
 	(segment
-		(start 29.447721 24.802028)
-		(end 35.702721 18.547028)
+		(start 38.35 19.45)
+		(end 39.35 18.45)
 		(width 0.5)
 		(layer "In2.Cu")
@@
 	)
 	(segment
+		(start 37.45 12.1)
+		(end 36.05 12.1)
+		(width 0.5)
+		(layer "F.Cu")
+		(net 11)
+	)
+	(segment
 		(start 55.217721 6.171176)
 		(end 55.217721 4.582028)
@@
 	)
 	(segment
-		(start 37.075 10.425)
-		(end 35.75 11.75)
-		(width 0.5)
-		(layer "F.Cu")
-		(net 11)
-	)
-	(segment
 		(start 62.962721 6.760326)
 		(end 61.873047 7.85)
@@
 	)
 	(segment
-		(start 35.75 11.75)
+		(start 36.05 12.1)
 		(end 35.75 11.8)
 		(width 0.5)
@@
 	)
 	(via
-		(at 37.075 10.425)
+		(at 37.45 12.1)
 		(size 0.75)
 		(drill 0.5)
@@
 	)
 	(segment
-		(start 95.472721 4.927028)
-		(end 94.347721 3.802028)
+		(start 38.75 12.1)
+		(end 39.6 12.95)
 		(width 0.5)
 		(layer "In2.Cu")
@@
 	)
 	(segment
-		(start 95.722721 4.927028)
-		(end 95.472721 4.927028)
+		(start 37.45 12.1)
+		(end 38.75 12.1)
 		(width 0.5)
 		(layer "In2.Cu")
@@
 	)
 	(segment
-		(start 48.924749 10.875)
-		(end 55.997721 3.802028)
+		(start 95.472721 4.927028)
+		(end 94.347721 3.802028)
+		(width 0.5)
+		(layer "In2.Cu")
+		(net 11)
+	)
+	(segment
+		(start 95.722721 4.927028)
+		(end 95.472721 4.927028)
 		(width 0.5)
 		(layer "In2.Cu")
@@
 	)
 	(segment
+		(start 55.997721 4.365452)
+		(end 55.997721 3.802028)
+		(width 0.5)
+		(layer "In2.Cu")
+		(net 11)
+	)
+	(segment
 		(start 63.997721 3.802028)
 		(end 55.997721 3.802028)
@@
 	)
 	(segment
-		(start 37.075 10.425)
-		(end 37.525 10.875)
+		(start 96.747721 5.952028)
+		(end 95.722721 4.927028)
 		(width 0.5)
 		(layer "In2.Cu")
@@
 	)
 	(segment
-		(start 96.747721 5.952028)
-		(end 95.722721 4.927028)
+		(start 47.413173 12.95)
+		(end 55.997721 4.365452)
 		(width 0.5)
 		(layer "In2.Cu")
@@
 	)
 	(segment
-		(start 37.525 10.875)
-		(end 48.924749 10.875)
+		(start 39.6 12.95)
+		(end 47.413173 12.95)
 		(width 0.5)
 		(layer "In2.Cu")
