File: 21xt/04-accessory-test/MAX5719_breakout/MAX5719_breakout.kicad_pcb (KiCad board)
At the start: 2 copper layers, 50 x 50 mm, 11 parts, among them IC1 MAX5719GSD+, J1 Conn_01x01, J2 Conn_01x02, J3 Conn_01x05, U1 TXB0104PWR

Commit message: finish max5719 breakout board
Parts:
- moved J1 1.27 mm to (164.8, 103.0)
- moved J2 1.27 mm to (172.4, 103.0)
Routing:
- net AOUT: track 8.79 -> 10.1 mm
- net 5v: track 26.7 -> 28.0 mm
Changed lines of the file:
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@@
 	(footprint "Connector_PinHeader_2.54mm:PinHeader_1x02_P2.54mm_Vertical"
 		(layer "F.Cu")
-		(at 172.44 104.28 -90)
+		(at 172.44 103.01 -90)
 		(descr "Through hole straight pin header, 1x02, 2.54mm pitch, single row")
 		(tags "Through hole pin header THT 1x02 2.54mm single row")
@@
 	(footprint "Connector_PinHeader_2.54mm:PinHeader_1x01_P2.54mm_Vertical"
 		(layer "F.Cu")
-		(at 164.82 104.28)
+		(at 164.82 103.01)
 		(descr "Through hole straight pin header, 1x01, 2.54mm pitch, single row")
 		(tags "Through hole pin header THT 1x01 2.54mm single row")
@@
 	)
 	(segment
-		(start 162.9105 112.13)
-		(end 159.17 112.13)
+		(start 171.12 108.97)
+		(end 169.9 107.75)
 		(width 0.2)
 		(layer "F.Cu")
@@
 	)
 	(segment
-		(start 167.3955 115.74)
-		(end 171.12 112.0155)
+		(start 169.9 107.75)
+		(end 169.9 103.01)
 		(width 0.2)
 		(layer "F.Cu")
@@
 	)
 	(segment
-		(start 169.9 107.75)
-		(end 171.12 108.97)
+		(start 162.9105 112.13)
+		(end 159.17 112.13)
 		(width 0.2)
 		(layer "F.Cu")
@@
 	)
 	(segment
-		(start 172.382 110.66)
-		(end 171.12 109.398)
+		(start 167.3955 115.74)
+		(end 171.12 112.0155)
 		(width 0.2)
 		(layer "F.Cu")
@@
 	)
 	(segment
-		(start 171.12 109.398)
-		(end 171.12 108.97)
+		(start 172.382 110.66)
+		(end 171.12 109.398)
 		(width 0.2)
 		(layer "F.Cu")
@@
 	)
 	(segment
-		(start 169.9 104.28)
-		(end 169.9 107.75)
+		(start 171.12 109.398)
+		(end 171.12 108.97)
 		(width 0.2)
 		(layer "F.Cu")
@@
 	)
 	(segment
-		(start 164.82 110.2295)
-		(end 166.5205 111.93)
+		(start 166.5205 111.93)
+		(end 164.82 110.2295)
 		(width 0.2)
 		(layer "F.Cu")
@@
 	)
 	(segment
-		(start 166.5205 111.93)
-		(end 166.958 111.93)
+		(start 166.958 111.93)
+		(end 166.5205 111.93)
 		(width 0.2)
 		(layer "F.Cu")
@@
 	)
 	(segment
-		(start 164.82 104.28)
-		(end 164.82 110.2295)
+		(start 164.82 110.2295)
+		(end 164.82 103.01)
 		(width 0.2)
 		(layer "F.Cu")

Commit message: stuff sorry im tired
Parts:
- removed C2: .1uF, Capacitor_SMD:C_0603_1608Metric
- removed U1: TXB0104PWR, accessory_test:TXB0104PWR
- added IC2: SN74LVC245ANSR, temp_deleteme:SOIC127P780X200-20N, F.Cu at (159.5, 113.5)
- added J4: Conn_01x04, Connector_PinHeader_2.54mm:PinHeader_1x04_P2.54mm_Vertical, F.Cu at (144.4, 110.6)
- J3: value Conn_01x05 -> Conn_01x03; footprint Connector_PinHeader_2.54mm:PinHeader_1x05_P2.54mm_Vertical -> Connector_PinHeader_2.54mm:PinHeader_1x03_P2.54mm_Vertical
- moved J3 21.8 mm to (157.1, 125.9), turned to 90 degrees
Connections:
- net 5v renamed 5vA
- J3 pad 1: 3v3 -> OE*
- J3 pad 2: CS -> 5vL
- J3 pad 3: SCLK -> DIR
Routing:
- net 3v3: track 19.0 -> 0.00 mm
- net OE*: track 0.00 -> 9.80 mm
- net GND: track 0.00 -> 8.89 mm
- net 5vA: track 28.0 -> 19.1 mm
- net 5vL: track 0.00 -> 8.39 mm
- net DIR: track 0.00 -> 7.23 mm
- net Net-(IC1-~{LDAC}): track 22.4 -> 17.2 mm
- net Net-(IC1-DIN): track 20.5 -> 16.1 mm
- net Net-(IC1-SCLK): track 15.7 -> 11.9 mm
- net Net-(IC1-~{CS}): track 10.1 -> 6.36 mm
- net MOSI: track 9.71 -> 13.0 mm
- net LDAC: track 10.5 -> 13.7 mm
- net SCLK: track 9.14 -> 11.9 mm
- net CS: track 9.92 -> 12.4 mm
Other:
- board text added: "5vA"
- board text added: "DAC"
- board text added: "LVL SHFTR"
- board text added: "OE* 5vL DIR"
- board text removed: "3v3"
- board text removed: "5v"

Commit message: v2 layout initial commit
Other:
- board text added: "LDAC"
- board text removed: "MISO"
Changed lines of the file:
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@@
 		)
 	)
-	(gr_text "MISO"
+	(gr_text "LDAC"
 		(at 139.75 118.78 0)
 		(layer "F.SilkS")
