File: 21xt/01-accessory/accessory_v3/digital_processing.kicad_sch (KiCad schematic)
At the start: 20 parts, among them IC6 TXB0108PWR, Q1 BSS138, Q2 BSS138, T1 749013011

Commit message: prod
Connections:
- net 3v3 renamed 3v3_pre2
- net 3v3_pre2: no longer C12.1, IC6.10 (OE), IC6.2 (VCCA)
- new net 3v3_pre: C12.1, IC6.10 (OE), IC6.2 (VCCA)
