File: 21xt/in-shaft-wsg/in-shaft-wsg-mommy/Analog.kicad_sch (KiCad schematic)
At the start: 18 parts, among them IC1 AD8237ARMZ, IC4 ADS1120IRVAR, IC5 ADS1120IRVAR, IC6 AD8237ARMZ, U2 AD5626BRMZ, U3 AD5626BRMZ

Commit message: shafted
Parts:
- removed C11, C12: 10nF, Capacitor_SMD:C_0402_1005Metric, symbol Device:C
- removed C7: .1uF, Capacitor_SMD:C_0402_1005Metric, symbol Device:C
- removed IC4: ADS1120IRVAR, 21xt_footprints:QFN50P350X350X100-17N-D, symbol 21xt_symbols:ADS1120IRVAR
- removed IC6: AD8237ARMZ, 21xt_footprints:SOP65P490X110-8N, symbol 21xt_symbols:AD8237ARMZ
- removed R17, R20, R22, R6: 1k, Resistor_SMD:R_0402_1005Metric, symbol Device:R
- removed R21: 200k, Resistor_SMD:R_0402_1005Metric, symbol Device:R
- removed R23: 50k, Resistor_SMD:R_0402_1005Metric, symbol Device:R
- removed U2, U3: AD5626BRMZ, 21xt_footprints:AD5626, symbol 21xt_symbols:AD5626BRMZ
- added C1: .1uF, Capacitor_SMD:C_0402_1005Metric, symbol Device:C
- added C14, C16, C17, C2, C3: 0.1uF, Capacitor_SMD:C_0402_1005Metric, symbol Device:C
- added C15, C18: 10nF, Capacitor_SMD:C_0402_1005Metric, symbol Device:C
- added IC2: AD8237ARMZ, 21xt_footprints:AD8237ARMZ, symbol 21xt_symbols:AD8237ARMZ
- added IC3: AD5689RBCPZ-RL7, 21xt_footprints:AD5689RBCPZ-RL7, symbol 21xt_symbols:AD5689RBCPZ-RL7
- added IC6: ADS1120IRVAR, 21xt_footprints:QFN50P350X350X100-17N-D, symbol 21xt_symbols:ADS1120IRVAR
- added R10, R25, R26, R8: 1k, Resistor_SMD:R_0402_1005Metric, symbol Device:R
- added R11, R12: 50k, Resistor_SMD:R_0402_1005Metric, symbol Device:R
- added R9: 200k, Resistor_SMD:R_0402_1005Metric, symbol Device:R
- C13: value .1uF -> 0.1uF
- IC1: footprint 21xt_footprints:SOP65P490X110-8N -> 21xt_footprints:AD8237ARMZ
- R5: value 200k -> 100
- R7: value 50k -> 200k
Connections:
- net DAC Bias is gone; now on net AmplifiedSig2: R7.2
- net 2V5 Lin: now also IC2.6 (REF), R10.1, R8.1
- net 3V3: now also C13.1, C16.1, IC3.14 (RSTSEL), IC3.8 (GAIN), IC3.9 (VLOGIC), IC6.11 (DVDD)
- net 5V Lin: now also C1.1, C2.2, C3.2, IC2.1 (BW), IC2.5 (+VS), IC3.3 (VDD); no longer C13.2
- net 5V Reference: now also R5.1, IC6.7 (REFP0)
- net 5V5: now also C14.1, C17.1, IC6.10 (AVDD)
- net ADC DReady1: now also IC6.12 (~{DRDY})
- net AmplifiedSig1: now also IC2.8 (VOUT), R26.1, R9.2; no longer IC1.8 (VOUT), R5.2
- net AmplifiedSig2: now also IC1.8 (VOUT), R25.1
- net CS-ADC1: now also IC6.16 (~{CS})
- net DAC Bias1: now also IC3.1 (VOUTA), IC6.5 (AIN2), R12.2
- net DAC Bias2: now also IC3.5 (VOUTB), R11.2
- net FilteredSig1: now also C18.1, IC6.8 (AIN1), R26.2
- net FilteredSig2: now also C15.1, R25.2
- net GNDA: now also C13.2, IC5.17 (EP), C1.2, C14.2, C15.2, C16.2, C17.2, C18.2, C2.1, C3.1, IC2.4 (-VS), IC3.17 (GND_2), IC3.2 (GND_1), IC6.17 (EP), IC6.3 (AVSS), IC6.4 (AIN3/REFN1), IC6.6 (REFN0); no longer C13.1
- net GNDD: now also IC6.2 (DGND)
- net Gage Excitation: now also IC6.9 (AIN0/REFP1)
- net MISO_ADC1: now also IC6.13 (DOUT/~{DRDY})
- net MOSI_ADC1: now also IC6.14 (DIN)
- net MOSI_DAC: now also IC3.12 (SDIN)
- net S1+: now also IC2.2 (+IN); no longer IC1.2 (+IN)
- net S1-: now also IC2.3 (-IN); no longer IC1.3 (-IN)
- net S2+: now also IC1.2 (+IN)
- net S2-: now also IC1.3 (-IN)
- net SCLK_ADC1: now also IC6.15 (SCLK)
- net SCLK_DAC: now also IC3.10 (SCLK)
- net at IC1.7 (FB), R7.1: now also R11.1, R8.2; no longer R5.1
- new net: IC3.15 (VREF), R5.2
- new net: IC2.7 (FB), R10.2, R12.1, R9.1
- new net CS-DAC: IC3.11 (~{SYNC})
- new net LDAC-DAC: IC3.7 (~{LDAC})
- no-connect marks 4 -> 6
Other:
- note removed: "dac"
