File: 21xt/in-shaft-wsg/in-shaft-wsg-mommy/References.kicad_sch (KiCad schematic)
At the start: 15 parts, among them IC3 MCP1502T-50E_CHY

Commit message: shafted
Parts:
- removed C1, C2: 10uF, Capacitor_SMD:C_0402_1005Metric, symbol Device:C
- removed C3: 1uF, Capacitor_SMD:C_0402_1005Metric, symbol Device:C
- removed IC3: MCP1502T-50E_CHY, 21xt_footprints:SOT95P280X145-6N, symbol 21xt_symbols:MCP1501T-50E_CHY
- removed R18: 806k, Resistor_SMD:R_0402_1005Metric, symbol Device:R
- removed R19: 80.6k, Resistor_SMD:R_0402_1005Metric, symbol Device:R
- added C11, C7: 1uF, Capacitor_SMD:C_0402_1005Metric, symbol Device:C
- added C12: 47uF, Capacitor_SMD:C_0805_2012Metric, symbol Device:C
- added IC4: MCP1502T-50E_CHY, 21xt_footprints:SOT95P280X145-6N, symbol 21xt_symbols:MCP1501T-50E_CHY
- added R22: 806k, Resistor_SMD:R_0402_1005Metric, symbol Device:R
- added R23: 80.6k, Resistor_SMD:R_0402_1005Metric, symbol Device:R
- C10: value 47uF -> 1uF; footprint Capacitor_SMD:C_0805_2012Metric -> Capacitor_SMD:C_0402_1005Metric
- C4: value 1uF -> 0.1uF
- C5, C6: value 1uF -> 10uF
- C8: value 0.1uF -> 1uF
Connections:
- net 2V5 Lin: now also C5.1, C7.1
- net 5V Lin: now also C6.1, C8.1; no longer C4.1
- net 5V Reference: now also IC4.1 (OUT)
- net 5V5: now also C4.1, C11.1, C12.1, IC4.4 (~{SHDN}), IC4.6 (VDD), R22.2; no longer C5.1, C6.1, C8.1
- net GNDA: now also C10.2, C8.2, C11.2, C7.2, IC4.2 (GND_1), IC4.3 (GND_2); no longer C4.2
- net GNDD: now also C4.2, C12.2, IC4.5 (GND_3), R23.1; no longer C10.2, C8.2
- net at PS3.5 (FB): now also R22.1, R23.2
