File: 21xt/02-mainbox/mainbox3.0/Pi5.kicad_sch (KiCad schematic)
At the start: 8 parts, among them IC1 SN74LVC2T45DCTTG4, J1 Conn_01x10, J12 Conn_02x20_Odd_Even

Commit message: main3.0
Parts:
- J12: footprint Connector_PinHeader_2.54mm:PinHeader_2x20_P2.54mm_Vertical -> RPi5Conn:PinHeader_2x20_P2.54mm_Vertical
Changed lines of the file:
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@@
 			)
 		)
-		(property "Footprint" "Connector_PinHeader_2.54mm:PinHeader_2x20_P2.54mm_Vertical"
+		(property "Footprint" "RPi5Conn:PinHeader_2x20_P2.54mm_Vertical"
 			(at 170.18 127 0)
 			(effects

Commit message: resolved error
Connections:
- net 3V3: no longer R10.2
- new net 3V3_XBEE: R10.2
Changed lines of the file:
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@@
 		)
 	)
-	(global_label "3V3"
+	(global_label "3V3_XBEE"
 		(shape input)
 		(at 210.82 121.92 270)
@@
 		)
 		(property "Intersheetrefs" "${INTERSHEET_REFS}"
-			(at 210.82 128.4128 90)
+			(at 210.82 134.1579 90)
 			(effects
 				(font
