File: 21xt/dyno_inst/dyno_inst_3/analogFE.kicad_sch (KiCad schematic)
At the start: 56 parts, among them U12 1SS362FV_L3F, U13 1SS362FV_L3F, U14 ADA4807-2ARM, U16 AD8429ARZ-R7, U17 1SS362FV_L3F, U18 1SS362FV_L3F, U19 ADA4807-1, U3 AD7175-2BRUZ

Commit message: layout done i think
Connections:
- net 3V3Ext renamed 3v3Ext
Changed lines of the file:
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@@
 		)
 	)
-	(global_label "3V3Ext"
+	(global_label "3v3Ext"
 		(shape input)
 		(at 194.31 71.12 180)
@@
 		)
 		(property "Intersheetrefs" "${INTERSHEET_REFS}"
-			(at 184.9144 71.12 0)
+			(at 185.0354 71.12 0)
 			(effects
 				(font
