File: 21xt/dyno_inst/dyno_inst_3/dyno_inst_3.kicad_pcb (KiCad board)
At the start: 4 copper layers, 86.1 x 99.8 mm, 140 parts, among them IC1 MCP1502T-25E_CHY, IC2 TC7660SEOA713, IC3 MCP1502T-25E_CHY, J1 Conn_01x05, J2 Conn_01x10, J3 Conn_01x03, J4 Barrel_Jack, J5 Conn_01x06, J6 Conn_01x04, J7 Conn_01x04, T1 749013011, U1 MAX14931FASE+, U10 LT3032IDE-5-TRPBF, U11 MAX14930FASE+, U12 1SS362FV_L3F, U13 1SS362FV_L3F, U14 ADA4807-2ARM, U16 AD8429ARZ-R7, U17 1SS362FV_L3F, U18 1SS362FV_L3F, U19 ADA4807-1, U2 MAX14930FASE+, U21 CME0303S3C, U23 CPC1017N, U24 LT3032IDE-5-TRPBF, U3 AD7175-2BRUZ, U4 DEV-16771, U5 LT3032IDE-5-TRPBF, U6 1S4E_1.5U, U7 1S4E_1.5U, U8 TL431DBZ, U9 TL431DBZ

Commit message: asdfdsf
Parts:
- moved CR5 4.05 mm to (191.2, 92.0)
- moved R40 2.81 mm to (194.8, 93.3), turned to 180 degrees
- moved U12 1.18 mm to (190.4, 106.0), turned to -90 degrees
- moved C79 0.40 mm to (171.7, 88.9)
Routing:
- net -5vcla: track 0.00 -> 56.0 mm, vias 0 -> 5
- net +5vcla: track 0.00 -> 46.3 mm, vias 0 -> 5
- net +5vexc: track 0.00 -> 28.1 mm
- net -5vexc: track 0.00 -> 24.0 mm
- net ACSIG^: track 0.00 -> 13.2 mm
- net +DCSIG^: track 0.00 -> 10.8 mm
- net -DCSIG^: track 0.00 -> 10.5 mm
- net +12v: track 2.86 -> 10.8 mm
- net GNDA: track 0.00 -> 5.76 mm
- net Net-(U10-OUTN): track 0.00 -> 5.61 mm
- net -DCSIG: track 0.00 -> 5.20 mm
- net +DCSIG: track 0.00 -> 5.02 mm
- net ACSIG: track 0.00 -> 4.36 mm
- net Net-(U12-C1/A2): track 0.00 -> 3.83 mm
- net Net-(U13-C1/A2): track 0.00 -> 3.78 mm
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- added copper zone on In1.Cu, net GNDA
Other:
- board text removed: "For Instructional Use Only."
- board text removed: "SOLIDWORKS Educational Product."

Commit message: i think i accidentally added some power distro stuff lol
Parts:
- moved C25 78.7 mm to (190.9, 63.6)
- moved J2 8.92 mm to (167.0, 42.2)
- moved C21 7.29 mm to (157.6, 91.7)
- moved C22 6.04 mm to (157.6, 90.7), turned to 180 degrees
- moved U2 3.79 mm to (155.2, 54.4)
- moved C1 3.79 mm to (151.4, 58.8)
- moved C4 3.79 mm to (151.4, 49.9)
- moved C19 3.29 mm to (160.7, 90.7), turned to 0 degrees
- moved R37 2.55 mm to (162.4, 110.8), turned to 0 degrees
- moved C27 1.59 mm to (155.9, 87.7), turned to -90 degrees
- moved C30 1.29 mm to (162.5, 97.9)
- moved R10 1.29 mm to (166.1, 94.7)
- moved U9 1.29 mm to (163.5, 95.5)
- moved R6 1.29 mm to (160.8, 94.8)
- moved R8 1.29 mm to (162.5, 93.1)
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Routing:
- net +5vref: track 1.97 -> 79.8 mm, vias 0 -> 6
- net -5vref: track 0.00 -> 65.0 mm, vias 0 -> 6
- net ACSHCAL: track 0.00 -> 64.1 mm, vias 0 -> 3
- net GNDA: track 5.76 -> 55.2 mm, vias 0 -> 47
- net ACSIG^: track 13.2 -> 54.5 mm
- net SE_DCSIG_filt: track 0.00 -> 27.8 mm
- net 3v3Ext: track 0.00 -> 24.9 mm, vias 0 -> 2
- net +12v: track 10.8 -> 31.1 mm, vias 0 -> 2
- net -5vexc: track 24.0 -> 43.6 mm
- net -2v5ref: track 3.48 -> 22.3 mm
- net -2v5adc: track 3.23 -> 19.1 mm
- net -12v: track 2.73 -> 18.4 mm, vias 0 -> 3
- net +2v5ref: track 2.76 -> 17.1 mm
- net BMISO: track 0.00 -> 12.9 mm
- net BSCLK: track 0.00 -> 12.2 mm
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- added copper zone on In2.Cu, net +12v
- added copper zone on In2.Cu, net -12v

Commit message: layout done i think
Parts:
- removed C88: 1uF, Capacitor_SMD:C_0603_1608Metric
- moved R45 0.70 mm to (135.1, 43.8), turned to 90 degrees
Connections:
- C10 pad 1: GNDA -> GND1
- C11 pad 1: GNDA -> GND1
- C12 pad 1: GNDA -> GND1
- C13 pad 1: GNDA -> GND1
- C14 pad 2: GNDA -> GND1
- C15 pad 2: GNDA -> GND1
- C17 pad 1: GNDA -> GND1
- C19 pad 1: GNDA -> GND1
- C22 pad 1: GNDA -> GND1
- C23 pad 1: GNDA -> GND1
- C24 pad 1: GNDA -> GND1
- C26 pad 2: GNDA -> GND1
- C27 pad 1: GNDA -> GND1
- C28 pad 1: GNDA -> GND1
- C29 pad 1: GNDA -> GND1
- C30 pad 1: GNDA -> GND1
- C31 pad 1: GNDD -> GND1
- C32 pad 1: GNDA -> GND1
- C33 pad 2: GNDD -> GND1
- C34 pad 2: GNDA -> GND1
- C35 pad 1: GNDA -> GND1
- C38 pad 1: GNDA -> GND1
- C39 pad 2: GNDA -> GND1
- C40 pad 1: GNDA -> GND1
- C41 pad 2: GNDA -> GND1
- C43 pad 1: GNDD -> GND1
- C44 pad 1: GNDD -> GND1
- C45 pad 1: GNDA -> GND1
- C47 pad 2: GNDA -> GND1
- C5 pad 1: 3V3Ext -> 3v3Ext
- C5 pad 2: GNDD -> GND1
- C53 pad 2: GNDA -> GND1
- C57 pad 2: GNDA -> GND1
- C58 pad 2: GNDA -> GND1
- C6 pad 1: 3V3Ext -> 3v3Ext
- C6 pad 2: GNDD -> GND1
- C61 pad 2: GNDA -> GND1
- C63 pad 2: GNDA -> GND1
- C69 pad 1: GNDPWR -> GND1
- C7 pad 1: GNDA -> GND1
- C70 pad 1: GNDPWR -> GND1
- C75 pad 2: GNDA -> GND1
- C76 pad 2: GNDA -> GND1
- C77 pad 2: GNDA -> GND1
- C78 pad 2: GNDA -> GND1
- C79 pad 1: GNDA -> GND1
- C8 pad 1: GNDA -> GND1
- C82 pad 1: GNDA -> GND1
- C83 pad 2: GNDA -> GND1
- C84 pad 1: GNDA -> GND1
- C87 pad 1: GNDPWR -> GND1
- C9 pad 1: GNDA -> GND1
- H1 pad 1: GND1 -> GND3
- H2 pad 1: GNDPWR -> GND1
- H4 pad 1: GND2 -> GND1
- IC1 pad 2: GNDA -> GND1
- IC1 pad 3: GNDA -> GND1
- IC1 pad 5: GNDA -> GND1
- IC2 pad 3: GNDPWR -> GND1
- IC3 pad 2: GNDA -> GND1
- IC3 pad 3: GNDA -> GND1
- IC3 pad 5: GNDA -> GND1
- J4 pad 2: GNDPWR -> GND1
- J7 pad 1: Rx+ -> Tx+
- J7 pad 4: Tx+ -> Rx+
- R10 pad 2: GNDA -> GND1
- R39 pad 1: GNDD -> GND1
- R9 pad 2: GNDA -> GND1
- U1 pad 15: GNDD -> GND1
- U1 pad 9: GNDD -> GND1
- U10 pad 10: GNDA -> GND1
- U10 pad 15: GNDA -> GND1
- U10 pad 4: GNDA -> GND1
- U10 pad 5: GNDA -> GND1
- U16 pad 6: GNDA -> GND1
- U21 pad 3: GNDD -> GND1
- U24 pad 10: GNDA -> GND1
- U24 pad 15: GNDA -> GND1
- U24 pad 4: GNDA -> GND1
- U24 pad 5: GNDA -> GND1
- U3 pad 15: GNDD -> GND1
- U3 pad 16: 3V3Ext -> 3v3Ext
- U3 pad 17: GNDD -> GND1
- U4 pad 30: Benc3 -> Benc1
- U4 pad 32: Benc1 -> Benc3
- U5 pad 10: GNDA -> GND1
- U5 pad 15: GNDA -> GND1
- U5 pad 4: GNDA -> GND1
- U5 pad 5: GNDA -> GND1
- U6 pad 1: GNDPWR -> GND1
- U7 pad 1: GNDPWR -> GND1
- U8 pad 1: GNDA -> GND1
- U9 pad 1: GNDA -> GND1
Routing:
- net GND1: track 6.09 -> 78.8 mm, vias 6 -> 67
- net GNDA: track 55.2 -> 0.00 mm, vias 47 -> 0
- net ASCLK: track 0.00 -> 51.8 mm
- net AMISO: track 0.00 -> 35.8 mm
- net AMOSI: track 0.00 -> 31.8 mm
- net Benc1: track 0.00 -> 26.5 mm
- net !ACS: track 0.00 -> 25.9 mm
- net Benc2: track 0.00 -> 24.0 mm
- net 3v3Teensy: track 3.33 -> 27.3 mm, vias 0 -> 4
- net Td-: track 0.00 -> 21.5 mm
- net GND3: track 3.57 -> 25.0 mm, vias 0 -> 14
- net Benc3: track 0.00 -> 21.4 mm
- net Td+: track 0.00 -> 21.4 mm
- net PWM: track 0.00 -> 20.1 mm
- net INB: track 0.00 -> 20.1 mm
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- added copper zone on In2.Cu, net 3v3Teensy
- added copper zone on In2.Cu, net 5venc
- added copper zone on In2.Cu, net 5vpwr
- removed copper zone on In1.Cu, net GNDA
- removed copper zone on In1.Cu, net GNDD
- removed copper zone on In1.Cu, net GNDPWR
Other:
- board text added: "INA ENA PWM CS ENB INB 5V GND NC GND"
- board text added: "PWR GND"
- board text added: "small hbridge"
- board text removed: "GND NC GND 5v INB ENB CS PWM ENA INA"

Commit message: kyle taylor wuz here
Parts:
- H1, H2, H3, H4: footprint MountingHole:MountingHole_3mm_Pad -> dynoinst_fp:dyno_inst_hole
- moved U7 0.08 mm to (199.5, 74.9)
Routing:
- net GND1: track 78.8 -> 79.6 mm, vias 67 -> 68
Other:
- board text added: "GND 5v ENC1 ENC2 ENC3"
- board text removed: "i will board mount small hbridge here"

Commit message: nothing happened
Other:
- board text added: "kyle taylor hates making bushings"
Changed lines of the file:
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@@
 		(tags "Through hole pin header THT 1x04 2.54mm single row")
 		(property "Reference" "U7"
-			(at 0 -2.33 360)
+			(at 0 -2.33 0)
 			(layer "F.SilkS")
 			(effects
@@
 		)
 		(property "Value" "1S4E_1.5U"
-			(at 0 9.95 360)
+			(at 0 9.95 0)
 			(layer "F.Fab")
 			(effects
@@
 		(tags "Through hole pin header THT 1x04 2.54mm single row")
 		(property "Reference" "U6"
-			(at 0 -2.33 360)
+			(at 0 -2.33 0)
 			(layer "F.SilkS")
 			(effects
@@
 		)
 		(property "Value" "1S4E_1.5U"
-			(at 0 9.95 360)
+			(at 0 9.95 0)
 			(layer "F.Fab")
 			(effects
@@
 				(bold yes)
 			)
+			(justify left bottom)
+		)
+	)
+	(gr_text "kyle taylor hates making bushings"
+		(at 140.3 71.6 0)
+		(layer "F.SilkS")
+		(effects
+			(font
+				(size 1 1)
+				(thickness 0.125)
+				(bold yes)
+			)
