File: 21xt/small_hbridge/small_hbridge.kicad_pcb (KiCad board)
At the start: 2 copper layers, 85 x 52.5 mm, 19 parts, among them J1 Screw_Terminal_01x02, J2 Screw_Terminal_01x02, J4 Conn_01x10, U1 VNH5019ATR-E, U2 STD3NK100Z

Commit message: done
Parts:
- moved J4 10.6 mm to (153.5, 100.8)
- moved C3 6.07 mm to (181.1, 79.7)
- moved C4 6.07 mm to (181.1, 78.2)
- moved R10 6.07 mm to (160.5, 94.6)
- moved U2 6.07 mm to (176.5, 72.5)
- moved C2 6.07 mm to (159.4, 90.8)
- moved C5 6.07 mm to (178.1, 66.5)
- moved R1 6.07 mm to (161.7, 87.1)
- moved R2 6.07 mm to (161.7, 91.5)
- moved R3 6.07 mm to (161.7, 85.6)
- moved R4 6.07 mm to (161.7, 93.1)
- moved R5 6.07 mm to (161.7, 88.6)
- moved R6 6.07 mm to (161.7, 90.1)
- moved R7 6.07 mm to (164.0, 91.2)
- moved R8 6.07 mm to (157.4, 89.4)
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Routing:
- net OUTB: track 61.4 -> 54.8 mm
- net OUTA: track 46.5 -> 40.5 mm
- net VDD: track 27.7 -> 23.2 mm
- net ENA: track 14.5 -> 10.1 mm
- net INB: track 12.8 -> 8.36 mm
- net CURRSNS: track 13.7 -> 9.40 mm
- net INA: track 15.0 -> 10.7 mm
- net ENB: track 13.5 -> 9.29 mm
- net 12v: track 30.1 -> 26.3 mm
- net PWM: track 14.1 -> 10.6 mm
Other:
- board size 85 x 52.5 mm -> 70.6 x 47 mm
- board text removed: "figure it out"

Commit message: aaaaa
Parts:
- removed J2: Screw_Terminal_01x02, dynoinst_fp:CONN_4DB-P108-02_TEC
- added J3: Barrel_Jack, dynoinst_fp:CUI_PJ-037A, F.Cu at (190.2, 87.2)
- J1: footprint dynoinst_fp:CONN_4DB-P108-02_TEC -> dynoinst_fp:282837-2_TYC
- moved C4 14.8 mm to (166.4, 78.3), turned to -90 degrees
- moved C3 13.3 mm to (167.9, 78.3), turned to -90 degrees
- moved C5 12.8 mm to (182.9, 78.3), turned to 90 degrees
- moved J1 7.21 mm to (190.4, 93.0), turned to -90 degrees
- moved U2 4.24 mm to (176.9, 76.7), turned to -90 degrees
- moved J4 1.56 mm to (155.1, 100.8)
- moved R8 0.45 mm to (157.9, 89.4)
Routing:
- net OUTB: track 54.8 -> 34.0 mm
- net 12v: track 26.3 -> 18.0 mm
- net Net-(U1-CP): track 18.1 -> 25.7 mm
- net OUTA: track 40.5 -> 37.8 mm
- net INB: track 8.36 -> 6.77 mm
- net VDD: track 23.2 -> 21.6 mm
- net ENB: track 9.29 -> 7.90 mm
- net ENA: track 10.1 -> 8.92 mm
- net CURRSNS: track 9.40 -> 8.41 mm
- net PWM: track 10.6 -> 9.76 mm
- net 12v': track 46.4 -> 45.7 mm
Other:
- board size 70.6 x 47 mm -> 42.4 x 30.4 mm
- board text added: "12v GND"
