File: 21xt/01-accessory/pre_amplifier/power.kicad_sch (KiCad schematic)
At the start: 1 part, among them IC1 LT6658AHMSE-5#PBF

Commit message: Continued schematic
Parts:
- added C1: 1u, symbol Device:C
- added C2, C5, C6: 0.1u, symbol Device:C
- added C3, C4, C7: 10u, symbol Device:C
- added D1: D_Schottky, symbol Device:D_Schottky
Connections:
- net GND: now reaches IC1.1 (GND_1)
- net GND: now also IC1.17 (GND_4), IC1.2 (GND_2), IC1.6 (GND_3), C1.1, C2.1, C3.1, C4.1, C5.1, C6.1, C7.1
- net 5v_reful: now reaches IC1.10 (VIN2)
- net 5v_reful: now also IC1.11 (VIN1), IC1.12 (VOUT1_F), IC1.13 (VOUT1_S), IC1.7 (VOUT2_S), IC1.8 (VOUT2_F), IC1.9 (~{OD}), C3.2, C4.2, C5.2, C6.2, C7.2
- net 11v1_schott: now reaches IC1.14 (VIN)
- net 11v1_schott: now also D1.1 (K)
- net at IC1.3 (BYPASS): now also C1.2
- net at IC1.5 (NR): now also C2.2
- new net 11v1_bat: D1.2 (A)
- no-connect marks 0 -> 3
Other:
- note added: "11v1 (90 mA) -> 5v (200 mA) refulator"
- note added: "11v1 Reverse Polarity Protection"
- note added: "150 + 50 mA"
- note added: "50 mA"
- note added: "dc/dc refulator: 1) Strain Gauges (14 * 10 = 140 mA) 2) DAC 3) Switches"
- moved on the sheet: IC1

Commit message: Reviewed schematic
Parts:
- added C55, C57: 4.7u, symbol Device:C
- added C56: 10u, symbol Device:C
- added C58: 0.1u, symbol Device:C
- added L1: 10u, symbol Device:L
- added NT1: NetTie_2, symbol Device:NetTie_2
- added PS1: P7805B-500, 21xt_footprints:CONV_P7805B-500, symbol 21xt_symbols:P7805B-500
Connections:
- net 11v1_schott: now also C55.2, L1.1
- net GND renamed GNDA
- net GNDA: now also C55.1, C56.1, C57.1, C58.1, NT1.1
- new net: C57.2, L1.2, PS1.1 (+VIN)
- new net 5v_buck: C56.2, C58.2, PS1.3 (+VOUT)
- new net B-: NT1.2, PS1.2 (GND)
Other:
- note added: "11v1 (100+ mA) -> 5v (200 mA) refulator"
- note added: "11v1 (250+ mA) -> 5v (500 mA) refulator"
- note added: "https://www.cui.com/product/resource/p78b-500.pdf ^ for footprint assignments"
- note removed: "11v1 (90 mA) -> 5v (200 mA) refulator"
- moved on the sheet: C1, C2, C3, C4, C5, C6, C7, D1, IC1

Commit message: added footprints
Parts:
- IC1: footprint SOP50P490X110-17N -> pre_amp_footprint_lib:LT6658AHMSE_footprint
Changed lines of the file:
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@@
 			)
 		)
-		(property "Footprint" "SOP50P490X110-17N"
+		(property "Footprint" "pre_amp_footprint_lib:LT6658AHMSE_footprint"
 			(at 220.98 177.47 0)
 			(effects

Commit message: added footprints
Parts:
- IC1: footprint pre_amp_footprint_lib:LT6658AHMSE_footprint -> 21xt_footprints:LT6658AHMSE-2.5-PBF
Changed lines of the file:
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@@
 			)
 		)
-		(property "Footprint" "pre_amp_footprint_lib:LT6658AHMSE_footprint"
+		(property "Footprint" "21xt_footprints:LT6658AHMSE-2.5-PBF"
 			(at 220.98 177.47 0)
 			(effects

Commit message: assigned footprints
Parts:
- C1, C2, C5, C58, C6: footprint (none) -> Capacitor_SMD:C_0402_1005Metric
- C3, C4, C56, C7: footprint (none) -> Capacitor_SMD:C_0603_1608Metric
- C55, C57: footprint (none) -> Capacitor_SMD:C_1206_3216Metric
- D1: footprint (none) -> Diode_SMD:D_1206_3216Metric
- L1: footprint (none) -> Inductor_SMD:L_0603_1608Metric
- NT1: footprint (none) -> NetTie:NetTie-2_SMD_Pad0.5mm
Connections:
- net GNDA: now also IC1.EPAD (GND_4); no longer IC1.17 (GND_4)
Other:
- note added: "11v1 (250+ mA) -> 5v (500 mA) buck converter"
- note removed: "11v1 (250+ mA) -> 5v (500 mA) refulator"

Commit message: Sandra pcb layout sess
Connections:
- net 11v1_schott: now also C5.2, C6.2, C7.2, IC1.10 (VIN2), IC1.11 (VIN1), IC1.9 (~{OD})
- net 5v_reful: no longer C5.2, C6.2, C7.2, IC1.10 (VIN2), IC1.11 (VIN1), IC1.9 (~{OD})
