File: 21xt/deans_distro/2M_3F/2M_3F.kicad_pcb (KiCad board)
At the start: 6 copper layers, 31.2 x 28 mm, 5 parts, among them J1 Conn_01x02, J2 Conn_01x02, J3 Conn_01x02, J4 Conn_01x02, J5 Conn_01x02

Commit message: adf
Parts:
- moved J3 7.26 mm to (107.3, 42.6)
- moved J2 7.26 mm to (84.8, 42.6)
Routing:
- net Net-(J1-Pin_1): vias 38 -> 34
- net GND: vias 35 -> 31
Other:
- board size 31.2 x 28 mm -> 32.6 x 28 mm
