File: 21xt/in-shaft-wsg/in-shaft-wsg-daughter/in-shaft-wsg-daughter.kicad_pcb (KiCad board)
At the start: 4 copper layers, 20.3 x 53.5 mm, 19 parts, among them J1 tall_usb_female, J2 Conn_01x04, J3 Conn_01x04

Commit message: v2
Other:
- board text added: "V2"
Changed lines of the file:
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@@
 		(tags "connector wire 0.1sqmm")
 		(property "Reference" "J3"
-			(at 5.4 -2 360)
+			(at 5.4 -2 0)
 			(layer "F.SilkS")
 			(hide yes)
@@
 		)
 		(property "Value" "Conn_01x04"
-			(at 5.4 2 360)
+			(at 5.4 2 0)
 			(layer "F.Fab")
 			(effects
@@
 		)
 		(property "Footprint" "21xt_footprints:tall usb female"
-			(at 0 0 360)
+			(at 0 0 0)
 			(layer "F.Fab")
 			(hide yes)
@@
 		)
 		(property "Datasheet" "2171800001"
-			(at 0 0 360)
+			(at 0 0 0)
 			(layer "F.Fab")
 			(hide yes)
@@
 		)
 		(property "Description" ""
-			(at 0 0 360)
+			(at 0 0 0)
 			(layer "F.Fab")
 			(hide yes)
@@
 				(bold yes)
 			)
+			(justify left bottom mirror)
+		)
+	)
+	(gr_text "V2"
+		(at 13.4 48.35 0)
+		(layer "B.SilkS")
+		(effects
+			(font
+				(size 3 3)
+				(thickness 0.75)
+				(bold yes)
+			)
