File: 21xt/03-wireless_strain_gauge/usb_c_daughter/usb_c_daughter.kicad_pcb (KiCad board)
At the start: 2 copper layers, 8 x 17 mm, 3 parts, among them J1 USB_C_Plug_USB2.0, J3 Conn_01x03

Commit message: v2
Routing:
- net SHIELD: track 6.61 -> 7.41 mm, vias 10 -> 11
- net GND: vias 0 -> 1
- added copper zone on In1.Cu, net GND
- added copper zone on In2.Cu, net GND
Other:
- board size 8 x 17 mm -> 8 x 14 mm
- copper layers 2 -> 4

Commit message: daughter files
Other:
- board size 8 x 14 mm -> 10 x 14 mm
Changed lines of the file:
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@@
 	(gr_arc
 		(start 7.247317 1.5)
-		(mid 7.778582 1.720624)
-		(end 7.997312 2.252679)
+		(mid 7.779378 1.718723)
+		(end 8 2.25)
+		(stroke
+			(width 0.01)
+			(type default)
+		)
+		(layer "Edge.Cuts")
+	)
+	(gr_line
+		(start 8 14.75)
+		(end 8 10)
 		(stroke
 			(width 0.01)
@@
 	)
 	(gr_line
+		(start 8 2.25)
+		(end 8 6.5)
+		(stroke
+			(width 0.01)
+			(type default)
+		)
+		(layer "Edge.Cuts")
+	)
+	(gr_line
 		(start 1 15.5)
 		(end 0.75 15.5)
@@
 	)
 	(gr_line
-		(start 7.997312 2.252679)
-		(end 7.952669 14.752679)
+		(start 8 6.5)
+		(end 10 6.5)
+		(stroke
+			(width 0.01)
+			(type default)
+		)
+		(layer "Edge.Cuts")
+	)
+	(gr_line
+		(start 10 6.5)
+		(end 10 10)
 		(stroke
 			(width 0.01)
@@
 		(start 1 1.5)
 		(end 0.75 1.5)
+		(stroke
+			(width 0.01)
+			(type default)
+		)
+		(layer "Edge.Cuts")
+	)
+	(gr_line
+		(start 8 10)
+		(end 10 10)
 		(stroke
 			(width 0.01)
@@
 	)
 	(gr_arc
-		(start 7.952669 14.752679)
-		(mid 7.732056 15.281276)
+		(start 8 14.75)
+		(mid 7.756278 15.289718)
 		(end 7.202674 15.5)
 		(stroke
